File: hardware/dev-board/kicad/hierarchical_sheets/zoe-m8q.kicad_sch (KiCad schematic)
At the start: 16 parts, among them U5 ZOE-M8Q

Commit message: More RF Stuff Routed
Parts:
- added D?: SZESD9R3.3ST5G, Diode_SMD:D_SOD-923, symbol Device:D_Zener
- added J?: CONSMA020.062-G, SRAD-FC:CONSMA020.062-G, symbol Connector:Conn_Coaxial
Connections:
- net A3_GND: now also D?.2 (A), J?.2 (Ext)
- net RTC_O: now reaches U5.P$J8 (J8_RTC_0), Y?.1
- net RTC_I: now reaches U5.P$J7 (J7_RTC_I), Y?.2
- net RF_IN: now reaches U5.P$A4 (A4_RF_IN)
- net RF_IN: now also D?.1 (K), J?.1 (In)
Other:
- moved on the sheet: C?, U5, Y?
