File: hardware/dev-board/kicad/hierarchical_sheets/zoe-m8q.kicad_sch (KiCad schematic)
At the start: 35 parts, among them J1 CONSMA020.062-G, U5 ZOE-M8Q, Y1 32.768kHz

Commit message: finished GPSschematic
Parts:
- removed JP?: SolderJumper_2_Open, Jumper:SolderJumper-2_P1.3mm_Open_RoundedPad1.0x1.5mm, symbol Jumper:SolderJumper_2_Open
- removed R? (x2): 10K, symbol Device:R
- removed TP?: Header, Connector_PinHeader_2.54mm:PinHeader_1x01_P2.54mm_Vertical, symbol Connector:TestPoint
- added JP? (x2): SolderJumper_2_Open, Jumper:SolderJumper-2_P1.3mm_Open_RoundedPad1.0x1.5mm, symbol Jumper:SolderJumper_2_Open
- added JP?: SolderJumper_3_Open, Jumper:SolderJumper-3_P1.3mm_Bridged12_RoundedPad1.0x1.5mm, symbol Jumper:SolderJumper_3_Open
- added TP? (x4): Header, Connector_PinHeader_2.54mm:PinHeader_1x01_P2.54mm_Vertical, symbol Connector:TestPoint
Connections:
- net A3_GND: now also JP?.1 (A)
- net D_SEL: now also JP?.2 (C)
- net GPS_VCC: now also JP?.3 (B)
- net TIMEPULSE: now reaches U5.P$C3 (C3_TIMEPULSE)
- net TIMEPULSE: now also JP?.1 (A), JP?.2 (B), TP?.1
- net PIO15: now reaches U5.P$C6 (C6_PIO15)
- net PIO15: now also TP?.1
- net PIO14: now reaches U5.P$F6 (F6_PIO14)
- net PIO14: now also TP?.1
- net EXTINT: now reaches U5.P$G4 (G4_PIO13/EXTINT)
- net EXTINT: now also JP?.1 (A), JP?.2 (B), TP?.1
- net ~{RESET}: now reaches U5.P$J6 (J6_RESET_N)
- net ~{RESET}: now also TP?.1
- net C4_SAFEBOOT renamed ~{SAFEBOOT}
- net ~{SAFEBOOT}: no longer TP?.1
Other:
- note added: "not using external flash"
- note added: "~{RESET} is active low, internal pullup"
- note added: "~{SAFEBOOT} is active low, internal pullup"
- note removed: "C4_SAFEBOOT should be tied to ground for SPI"
- moved on the sheet: JP?, TP?

Commit message: file sync
Parts:
- JP?: footprint Jumper:SolderJumper-3_P1.3mm_Bridged12_RoundedPad1.0x1.5mm -> Jumper:SolderJumper-3_P1.3mm_Open_RoundedPad1.0x1.5mm
Changed lines of the file:
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@@
       (effects (font (size 1.27 1.27)) hide)
     )
-    (property "Footprint" "Jumper:SolderJumper-3_P1.3mm_Bridged12_RoundedPad1.0x1.5mm" (id 2) (at 201.93 156.845 0)
+    (property "Footprint" "Jumper:SolderJumper-3_P1.3mm_Open_RoundedPad1.0x1.5mm" (id 2) (at 201.93 156.845 0)
       (effects (font (size 1.27 1.27)) hide)
     )

Commit message: rf is hard
Parts:
- added TP21, TP32: Header, Connector_PinHeader_2.54mm:PinHeader_1x01_P2.54mm_Vertical, symbol Connector:TestPoint
- gave numbers to parts that had none: 20
Connections:
- net GPS_VCC: now also TP21.1
- net V_BCKP: now also TP32.1
Other:
- moved on the sheet: JP21, JP22, JP23, JP24, JP25, JP26, JP27, JP28, TP19, TP20, TP22, TP23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
