File: hardware/dev-board/kicad/hierarchical_sheets/_autosave-zoe-m8q.kicad_sch (KiCad schematic)
At the start: 35 parts, among them J1 CONSMA020.062-G, U5 ZOE-M8Q, Y1 32.768kHz

Commit message: more gps work
Connections:
- net C4_SAFEBOOT: no longer TP?.1, U5.P$C4 (C4_SAFEBOOT)
- new net SAFEBOOT: TP?.1, U5.P$C4 (C4_SAFEBOOT)
Changed lines of the file:
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@@
+    (stroke (width 0) (type default) (color 0 0 0 0))
+  )
+  (wire (pts (xy 59.69 64.77) (xy 70.485 64.77))
     (stroke (width 0) (type default) (color 0 0 0 0))
   )
@@
   )
   (wire (pts (xy 103.505 52.07) (xy 103.505 50.165))
-    (stroke (width 0) (type default) (color 0 0 0 0))
-  )
-  (wire (pts (xy 56.515 64.77) (xy 70.485 64.77))
     (stroke (width 0) (type default) (color 0 0 0 0))
   )
@@
     (effects (font (size 1.27 1.27)) (justify left bottom))
   )
-  (label "C4_SAFEBOOT" (at 56.515 64.77 0)
+  (label "SAFEBOOT" (at 59.69 64.77 0)
     (effects (font (size 1.27 1.27)) (justify left bottom))
   )
@@
     (effects (font (size 1.27 1.27)) (justify left bottom))
   )
-  (label "C4_SAFEBOOT" (at 236.855 127 180)
-    (effects (font (size 1.27 1.27)) (justify right bottom))
-  )
+  (label "SAFEBOOT" (at 236.855 127 180)
+    (effects (font (size 1.27 1.27)) (justify right bottom))
+  )
