File: hardware/dev-board/kicad/hierarchical_sheets/icm-20608g.kicad_sch (KiCad schematic)
At the start: 20 parts

Commit message: Update Files
Parts:
- gave numbers to parts that had none: 20
Changed lines of the file:
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@@
   (symbol (lib_id "Device:C_Small") (at 92.71 100.33 0) (unit 1)
     (in_bom yes) (on_board yes) (fields_autoplaced)
-    (property "Reference" "C?" (id 0) (at 95.25 99.0662 0)
+    (property "Reference" "C3" (id 0) (at 95.25 99.0662 0)
       (effects (font (size 1.27 1.27)) (justify left))
     )
@@
   (symbol (lib_id "Device:R") (at 182.88 111.76 90) (unit 1)
     (in_bom yes) (on_board yes)
-    (property "Reference" "R?" (id 0) (at 182.88 109.22 90))
+    (property "Reference" "R1" (id 0) (at 182.88 109.22 90))
     (property "Value" "10K" (id 1) (at 182.88 111.76 90))
     (property "Footprint" "" (id 2) (at 182.88 113.538 90)
@@
   (symbol (lib_id "Connector:TestPoint") (at 199.39 100.33 0) (unit 1)
     (in_bom yes) (on_board yes)
-    (property "Reference" "TP?" (id 0) (at 200.66 96.52 0)
+    (property "Reference" "TP6" (id 0) (at 200.66 96.52 0)
       (effects (font (size 1.27 1.27)) (justify left))
     )
@@
   (symbol (lib_id "Sensor_Motion:ICM-20602") (at 69.85 92.71 0) (unit 1)
     (in_bom yes) (on_board yes)
-    (property "Reference" "U?" (id 0) (at 53.34 77.47 0)
+    (property "Reference" "U1" (id 0) (at 53.34 77.47 0)
       (effects (font (size 1.27 1.27)) (justify left))
     )
@@
   (symbol (lib_id "Device:C_Small") (at 92.71 78.74 0) (unit 1)
     (in_bom yes) (on_board yes) (fields_autoplaced)
-    (property "Reference" "C?" (id 0) (at 95.25 77.4762 0)
+    (property "Reference" "C2" (id 0) (at 95.25 77.4762 0)
       (effects (font (size 1.27 1.27)) (justify left))
     )
@@
   (symbol (lib_id "Jumper:SolderJumper_2_Open") (at 183.515 68.58 0) (unit 1)
     (in_bom yes) (on_board yes)
-    (property "Reference" "JP?" (id 0) (at 183.515 66.04 0))
+    (property "Reference" "JP2" (id 0) (at 183.515 66.04 0))
     (property "Value" "SolderJumper_2_Open" (id 1) (at 183.515 64.77 0)
       (effects (font (size 1.27 1.27)) hide)
@@
   (symbol (lib_id "Connector:TestPoint") (at 199.39 67.31 0) (unit 1)
     (in_bom yes) (on_board yes)
-    (property "Reference" "TP?" (id 0) (at 200.66 63.5 0)
+    (property "Reference" "TP2" (id 0) (at 200.66 63.5 0)
       (effects (font (size 1.27 1.27)) (justify left))
     )
@@
   (symbol (lib_id "Device:C_Small") (at 82.55 78.74 0) (unit 1)
     (in_bom yes) (on_board yes) (fields_autoplaced)
-    (property "Reference" "C?" (id 0) (at 85.09 77.4762 0)
+    (property "Reference" "C1" (id 0) (at 85.09 77.4762 0)
       (effects (font (size 1.27 1.27)) (justify left))
     )
@@
   (symbol (lib_id "Jumper:SolderJumper_2_Open") (at 184.15 93.345 0) (unit 1)
     (in_bom yes) (on_board yes)
-    (property "Reference" "JP?" (id 0) (at 184.15 90.805 0))
+    (property "Reference" "JP5" (id 0) (at 184.15 90.805 0))
     (property "Value" "SolderJumper_2_Open" (id 1) (at 184.15 89.535 0)
       (effects (font (size 1.27 1.27)) hide)
@@
   (symbol (lib_id "power:GND") (at 69.85 106.68 0) (unit 1)
     (in_bom yes) (on_board yes)
-    (property "Reference" "#PWR?" (id 0) (at 69.85 113.03 0)
+    (property "Reference" "#PWR0103" (id 0) (at 69.85 113.03 0)
       (effects (font (size 1.27 1.27)) hide)
     )
@@
   (symbol (lib_id "power:+3V3") (at 166.37 57.785 0) (unit 1)
     (in_bom yes) (on_board yes) (fields_autoplaced)
-    (property "Reference" "#PWR?" (id 0) (at 166.37 61.595 0)
+    (property "Reference" "#PWR0102" (id 0) (at 166.37 61.595 0)
       (effects (font (size 1.27 1.27)) hide)
     )
@@
   (symbol (lib_id "power:GND") (at 172.72 113.665 0) (unit 1)
     (in_bom yes) (on_board yes) (fields_autoplaced)
-    (property "Reference" "#PWR?" (id 0) (at 172.72 120.015 0)
+    (property "Reference" "#PWR0104" (id 0) (at 172.72 120.015 0)
       (effects (font (size 1.27 1.27)) hide)
     )
@@
   (symbol (lib_id "Connector:TestPoint") (at 199.39 92.075 0) (unit 1)
     (in_bom yes) (on_board yes)
-    (property "Reference" "TP?" (id 0) (at 200.66 88.265 0)
+    (property "Reference" "TP5" (id 0) (at 200.66 88.265 0)
       (effects (font (size 1.27 1.27)) (justify left))
     )
@@
   (symbol (lib_id "Device:C_Small") (at 102.87 78.74 0) (unit 1)
     (in_bom yes) (on_board yes) (fields_autoplaced)
-    (property "Reference" "C?" (id 0) (at 105.41 77.4762 0)
+    (property "Reference" "C4" (id 0) (at 105.41 77.4762 0)
       (effects (font (size 1.27 1.27)) (justify left))
     )
@@
   (symbol (lib_id "Connector:TestPoint") (at 199.39 75.565 0) (unit 1)
     (in_bom yes) (on_board yes)
-    (property "Reference" "TP?" (id 0) (at 200.66 71.755 0)
+    (property "Reference" "TP3" (id 0) (at 200.66 71.755 0)
       (effects (font (size 1.27 1.27)) (justify left))
     )
@@
   (symbol (lib_id "Connector:TestPoint") (at 199.39 83.82 0) (unit 1)
     (in_bom yes) (on_board yes)
-    (property "Reference" "TP?" (id 0) (at 200.66 80.01 0)
+    (property "Reference" "TP4" (id 0) (at 200.66 80.01 0)
       (effects (font (size 1.27 1.27)) (justify left))
     )
@@
   (symbol (lib_id "Jumper:SolderJumper_2_Open") (at 183.515 85.09 0) (unit 1)
     (in_bom yes) (on_board yes)
-    (property "Reference" "JP?" (id 0) (at 183.515 82.55 0))
+    (property "Reference" "JP4" (id 0) (at 183.515 82.55 0))
     (property "Value" "SolderJumper_2_Open" (id 1) (at 183.515 81.28 0)
       (effects (font (size 1.27 1.27)) hide)
@@
   (symbol (lib_id "Connector:TestPoint") (at 199.39 123.19 0) (unit 1)
     (in_bom yes) (on_board yes)
-    (property "Reference" "TP?" (id 0) (at 200.66 119.38 0)
+    (property "Reference" "TP8" (id 0) (at 200.66 119.38 0)
       (effects (font (size 1.27 1.27)) (justify left))
     )
@@
   (symbol (lib_id "power:GND") (at 102.87 82.55 0) (unit 1)
     (in_bom yes) (on_board yes)
-    (property "Reference" "#PWR?" (id 0) (at 102.87 88.9 0)
+    (property "Reference" "#PWR0101" (id 0) (at 102.87 88.9 0)
       (effects (font (size 1.27 1.27)) hide)
     )
@@
   (symbol (lib_id "Jumper:SolderJumper_2_Open") (at 184.15 101.6 0) (unit 1)
     (in_bom yes) (on_board yes)
-    (property "Reference" "JP?" (id 0) (at 184.15 99.06 0))
+    (property "Reference" "JP6" (id 0) (at 184.15 99.06 0))
     (property "Value" "SolderJumper_2_Open" (id 1) (at 184.15 97.79 0)
       (effects (font (size 1.27 1.27)) hide)
@@
   (symbol (lib_id "Jumper:SolderJumper_2_Open") (at 183.515 60.325 0) (unit 1)
     (in_bom yes) (on_board yes)
-    (property "Reference" "JP?" (id 0) (at 183.515 57.785 0))
+    (property "Reference" "JP1" (id 0) (at 183.515 57.785 0))
     (property "Value" "SolderJumper_2_Open" (id 1) (at 183.515 56.515 0)
       (effects (font (size 1.27 1.27)) hide)
@@
   (symbol (lib_id "Connector:TestPoint") (at 199.39 109.855 0) (unit 1)
     (in_bom yes) (on_board yes)
-    (property "Reference" "TP?" (id 0) (at 200.66 106.045 0)
+    (property "Reference" "TP7" (id 0) (at 200.66 106.045 0)
       (effects (font (size 1.27 1.27)) (justify left))
     )
@@
   (symbol (lib_id "Jumper:SolderJumper_2_Open") (at 183.515 76.835 0) (unit 1)
     (in_bom yes) (on_board yes)
-    (property "Reference" "JP?" (id 0) (at 183.515 74.295 0))
+    (property "Reference" "JP3" (id 0) (at 183.515 74.295 0))
     (property "Value" "SolderJumper_2_Open" (id 1) (at 183.515 73.025 0)
       (effects (font (size 1.27 1.27)) hide)
@@
   (symbol (lib_id "Connector:TestPoint") (at 199.39 58.42 0) (unit 1)
     (in_bom yes) (on_board yes)
-    (property "Reference" "TP?" (id 0) (at 200.66 54.61 0)
-      (effects (font (size 1.27 1.27)) (justify left))
-    )
+    (property "Reference" "TP1" (id 0) (at 200.66 54.61 0)
+      (effects (font (size 1.27 1.27)) (justify left))
+    )

Commit message: rf is hard
Parts:
- removed R1: 10K, symbol Device:R
- added JP18: SolderJumper_3_Open, Jumper:SolderJumper-3_P1.3mm_Open_RoundedPad1.0x1.5mm, symbol Jumper:SolderJumper_3_Open
Connections:
- net +3V3: now also JP18.3 (B)
- net FSYNC: now also JP18.2 (C)
- net GND: now also JP18.1 (A)
Other:
- moved on the sheet: TP8
