File: hardware/dev-board/kicad/hierarchical_sheets/kx134-1211.kicad_sch (KiCad schematic)
At the start: 14 parts

Commit message: Update Files
Parts:
- gave numbers to parts that had none: 14
Changed lines of the file:
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@@
   (symbol (lib_id "Device:C_Small") (at 121.92 82.55 0) (unit 1)
     (in_bom yes) (on_board yes) (fields_autoplaced)
-    (property "Reference" "C?" (id 0) (at 125.095 81.2862 0)
+    (property "Reference" "C6" (id 0) (at 125.095 81.2862 0)
       (effects (font (size 1.27 1.27)) (justify left))
     )
@@
   (symbol (lib_id "power:+3V3") (at 169.545 67.31 0) (unit 1)
     (in_bom yes) (on_board yes) (fields_autoplaced)
-    (property "Reference" "#PWR?" (id 0) (at 169.545 71.12 0)
+    (property "Reference" "#PWR0108" (id 0) (at 169.545 71.12 0)
       (effects (font (size 1.27 1.27)) hide)
     )
@@
   (symbol (lib_id "power:GND") (at 95.25 111.76 0) (unit 1)
     (in_bom yes) (on_board yes)
-    (property "Reference" "#PWR?" (id 0) (at 95.25 118.11 0)
+    (property "Reference" "#PWR0109" (id 0) (at 95.25 118.11 0)
       (effects (font (size 1.27 1.27)) hide)
     )
@@
   (symbol (lib_id "Jumper:SolderJumper_2_Open") (at 194.945 82.55 0) (unit 1)
     (in_bom yes) (on_board yes)
-    (property "Reference" "JP?" (id 0) (at 194.945 80.01 0))
+    (property "Reference" "JP11" (id 0) (at 194.945 80.01 0))
     (property "Value" "SolderJumper_2_Open" (id 1) (at 194.945 78.74 0)
       (effects (font (size 1.27 1.27)) hide)
@@
   (symbol (lib_id "Jumper:SolderJumper_2_Open") (at 194.945 76.2 0) (unit 1)
     (in_bom yes) (on_board yes)
-    (property "Reference" "JP?" (id 0) (at 194.945 73.66 0))
+    (property "Reference" "JP10" (id 0) (at 194.945 73.66 0))
     (property "Value" "SolderJumper_2_Open" (id 1) (at 194.945 72.39 0)
       (effects (font (size 1.27 1.27)) hide)
@@
   (symbol (lib_id "Connector:TestPoint") (at 202.565 106.68 0) (unit 1)
     (in_bom yes) (on_board yes)
-    (property "Reference" "TP?" (id 0) (at 203.835 102.87 0)
+    (property "Reference" "TP10" (id 0) (at 203.835 102.87 0)
       (effects (font (size 1.27 1.27)) (justify left))
     )
@@
   (symbol (lib_id "Sensor_Motion:KX122-1042") (at 95.25 97.79 0) (unit 1)
     (in_bom yes) (on_board yes)
-    (property "Reference" "U?" (id 0) (at 78.74 82.55 0)
+    (property "Reference" "U2" (id 0) (at 78.74 82.55 0)
       (effects (font (size 1.27 1.27)) (justify left))
     )
@@
   (symbol (lib_id "power:GND") (at 118.11 109.22 0) (unit 1)
     (in_bom yes) (on_board yes)
-    (property "Reference" "#PWR?" (id 0) (at 118.11 115.57 0)
+    (property "Reference" "#PWR0105" (id 0) (at 118.11 115.57 0)
       (effects (font (size 1.27 1.27)) hide)
     )
@@
   (symbol (lib_id "Jumper:SolderJumper_2_Open") (at 194.945 88.9 0) (unit 1)
     (in_bom yes) (on_board yes)
-    (property "Reference" "JP?" (id 0) (at 194.945 86.36 0))
+    (property "Reference" "JP12" (id 0) (at 194.945 86.36 0))
     (property "Value" "SolderJumper_2_Open" (id 1) (at 194.945 85.09 0)
       (effects (font (size 1.27 1.27)) hide)
@@
   (symbol (lib_id "Connector:TestPoint") (at 202.565 97.79 0) (unit 1)
     (in_bom yes) (on_board yes)
-    (property "Reference" "TP?" (id 0) (at 203.835 93.98 0)
+    (property "Reference" "TP9" (id 0) (at 203.835 93.98 0)
       (effects (font (size 1.27 1.27)) (justify left))
     )
@@
   (symbol (lib_id "Connector:TestPoint") (at 202.565 128.27 0) (unit 1)
     (in_bom yes) (on_board yes)
-    (property "Reference" "TP?" (id 0) (at 203.835 124.46 0)
+    (property "Reference" "TP12" (id 0) (at 203.835 124.46 0)
       (effects (font (size 1.27 1.27)) (justify left))
     )
@@
   (symbol (lib_id "Device:R") (at 186.055 118.11 90) (unit 1)
     (in_bom yes) (on_board yes)
-    (property "Reference" "R?" (id 0) (at 186.055 115.57 90))
+    (property "Reference" "R2" (id 0) (at 186.055 115.57 90))
     (property "Value" "10K" (id 1) (at 186.055 118.11 90))
     (property "Footprint" "" (id 2) (at 186.055 119.888 90)
@@
   (symbol (lib_id "Jumper:SolderJumper_2_Open") (at 187.325 99.06 0) (unit 1)
     (in_bom yes) (on_board yes)
-    (property "Reference" "JP?" (id 0) (at 187.325 96.52 0))
+    (property "Reference" "JP7" (id 0) (at 187.325 96.52 0))
     (property "Value" "SolderJumper_2_Open" (id 1) (at 187.325 95.25 0)
       (effects (font (size 1.27 1.27)) hide)
@@
   (symbol (lib_id "Jumper:SolderJumper_2_Open") (at 194.945 69.85 0) (unit 1)
     (in_bom yes) (on_board yes)
-    (property "Reference" "JP?" (id 0) (at 194.945 67.31 0))
+    (property "Reference" "JP9" (id 0) (at 194.945 67.31 0))
     (property "Value" "SolderJumper_2_Open" (id 1) (at 194.945 66.04 0)
       (effects (font (size 1.27 1.27)) hide)
@@
   (symbol (lib_id "power:GND") (at 175.895 120.015 0) (unit 1)
     (in_bom yes) (on_board yes) (fields_autoplaced)
-    (property "Reference" "#PWR?" (id 0) (at 175.895 126.365 0)
+    (property "Reference" "#PWR0107" (id 0) (at 175.895 126.365 0)
       (effects (font (size 1.27 1.27)) hide)
     )
@@
   (symbol (lib_id "Device:C_Small") (at 111.76 82.55 0) (unit 1)
     (in_bom yes) (on_board yes) (fields_autoplaced)
-    (property "Reference" "C?" (id 0) (at 114.3 81.2862 0)
+    (property "Reference" "C5" (id 0) (at 114.3 81.2862 0)
       (effects (font (size 1.27 1.27)) (justify left))
     )
@@
   (symbol (lib_id "Connector:TestPoint") (at 202.565 116.205 0) (unit 1)
     (in_bom yes) (on_board yes)
-    (property "Reference" "TP?" (id 0) (at 203.835 112.395 0)
+    (property "Reference" "TP11" (id 0) (at 203.835 112.395 0)
       (effects (font (size 1.27 1.27)) (justify left))
     )
@@
   (symbol (lib_id "power:GND") (at 121.92 86.995 0) (unit 1)
     (in_bom yes) (on_board yes)
-    (property "Reference" "#PWR?" (id 0) (at 121.92 93.345 0)
+    (property "Reference" "#PWR0106" (id 0) (at 121.92 93.345 0)
       (effects (font (size 1.27 1.27)) hide)
     )
@@
   (symbol (lib_id "Jumper:SolderJumper_2_Open") (at 187.325 107.95 0) (unit 1)
     (in_bom yes) (on_board yes)
-    (property "Reference" "JP?" (id 0) (at 187.325 105.41 0))
+    (property "Reference" "JP8" (id 0) (at 187.325 105.41 0))
     (property "Value" "SolderJumper_2_Open" (id 1) (at 187.325 104.14 0)
       (effects (font (size 1.27 1.27)) hide)

Commit message: rf is hard
Parts:
- removed R2: 10K, symbol Device:R
- added JP19: SolderJumper_3_Open, Jumper:SolderJumper-3_P1.3mm_Open_RoundedPad1.0x1.5mm, symbol Jumper:SolderJumper_3_Open
Connections:
- net +3V3: now also JP19.3 (B)
- net GND: now also JP19.1 (A)
- net TRIG: now also JP19.2 (C)
Other:
- moved on the sheet: TP12
