File: hardware/dev-board/kicad/hierarchical_sheets/mmc5983ma.kicad_sch (KiCad schematic)
At the start: 1 part, among them U4 MMC5983MA

Commit message: file sync
Parts:
- added C?: 10nF, symbol Device:C_Small
Connections:
- net GND: now reaches U4.11 (GND), U4.12 (NC), U4.14 (NC), U4.3 (NC), U4.6 (NC), U4.7 (NC), U4.8 (NC), U4.9 (GND)
Changed lines of the file:
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@@
     (comment 1 "Seth Sievers")
+  )
+  (wire (pts (xy 144.78 111.125) (xy 144.78 112.395))
+    (stroke (width 0) (type default) (color 0 0 0 0))
+  )
+  (symbol (lib_id "Device:C_Small") (at 160.655 100.965 0) (unit 1)
+    (in_bom yes) (on_board yes) (fields_autoplaced)
+    (property "Reference" "C?" (id 0) (at 163.195 99.7012 0)
+      (effects (font (size 1.27 1.27)) (justify left))
+    )
+    (property "Value" "10nF" (id 1) (at 163.195 102.2412 0)
+      (effects (font (size 1.27 1.27)) (justify left))
+    )
+    (property "Footprint" "" (id 2) (at 160.655 100.965 0)
+      (effects (font (size 1.27 1.27)) hide)
+    )
+    (property "Datasheet" "~" (id 3) (at 160.655 100.965 0)
+      (effects (font (size 1.27 1.27)) hide)
+    )
+    (pin "1")
+    (pin "2")
+  )
+  (symbol (lib_id "power:GND") (at 144.78 112.395 0) (unit 1)
+    (in_bom yes) (on_board yes) (fields_autoplaced)
+    (property "Reference" "#PWR?" (id 0) (at 144.78 118.745 0)
+      (effects (font (size 1.27 1.27)) hide)
+    )
+    (property "Value" "GND" (id 1) (at 144.78 116.8384 0))
+    (property "Footprint" "" (id 2) (at 144.78 112.395 0)
+      (effects (font (size 1.27 1.27)) hide)
+    )
+    (property "Datasheet" "" (id 3) (at 144.78 112.395 0)
+      (effects (font (size 1.27 1.27)) hide)
+    )
+    (pin "1")
   )
   (symbol (lib_id "Sensor_Magnetic:MMC5883MA") (at 143.51 97.155 0) (unit 1)

Commit message: rf is hard
Parts:
- added C20: 10nF, symbol Device:C_Small
- added C22: 0.1μF, symbol Device:C_Small
- added JP? (x6): SolderJumper_2_Open, Jumper:SolderJumper-2_P1.3mm_Open_RoundedPad1.0x1.5mm, symbol Jumper:SolderJumper_2_Open
- added TP? (x6): Header, Connector_PinHeader_2.54mm:PinHeader_1x01_P2.54mm_Vertical, symbol Connector:TestPoint
- C21: renamed from C?; value 10nF -> 10μF
Connections:
- net GND: now also C21.2, C20.2, C22.2
- net CAP: now reaches C21.1
- net CAP: now also U4.10 (CAP)
- net SCK: now reaches U4.1 (SCL/SCK)
- net SCK: now also JP?.1 (A), JP?.2 (B), TP?.1
- net +3V3: now reaches U4.13 (VDDIO)
- net +3V3: now also U4.2 (VDD), C20.1, C22.1, JP?.1 (A), JP?.2 (B), TP?.1
- net INT: now reaches U4.15 (INT)
- net INT: now also JP?.1 (A), JP?.2 (B), TP?.1
- net MOSI: now reaches U4.16 (SDA/SDI)
- net MOSI: now also JP?.1 (A), JP?.2 (B), TP?.1
- net ~{CS}: now reaches U4.4 (~{CS})
- net ~{CS}: now also JP?.1 (A), JP?.2 (B), TP?.1
- net MISO: now reaches U4.5 (SDO)
- net MISO: now also JP?.1 (A), JP?.2 (B), TP?.1
Other:
- note added: "*Remove for final*"
- note added: "DEBUG"
- note added: "MMC5983MA"
- moved on the sheet: C21, U4
