File: hardware/dev-board/kicad/hierarchical_sheets/ms5611.kicad_sch (KiCad schematic)
At the start: 15 parts

Commit message: Update Files
Parts:
- gave numbers to parts that had none: 15
Other:
- company: (none) -> Missouri S&T Rocket Design Team
- title: (none) -> Barometer
- moved on the sheet: C7, C8, JP13, JP14, JP15, JP16, JP17, R3, TP13, TP14, TP15, TP16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

Commit message: rf is hard
Parts:
- removed R3: 10K, symbol Device:R
- added JP20: SolderJumper_3_Open, Jumper:SolderJumper-3_P1.3mm_Open_RoundedPad1.0x1.5mm, symbol Jumper:SolderJumper_3_Open
- U3: Digikey (none) -> https://www.digikey.com/en/products/detail/te-connectivity-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
Connections:
- net +3V3: now also JP20.3 (B)
- net GND: now also JP20.1 (A)
- net PS: now also JP20.2 (C)
Other:
- note added: "PS should be tied to ground for SPI"
- note removed: "Tie PS to ground for SPI"
Changed lines of the file:
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@@
   (junction (at 129.54 85.725) (diameter 0) (color 0 0 0 0)
   )
-  (junction (at 199.39 109.855) (diameter 0) (color 0 0 0 0)
-  )
   (junction (at 199.39 84.455) (diameter 0) (color 0 0 0 0)
   )
@@
   (junction (at 129.54 78.105) (diameter 0) (color 0 0 0 0)
   )
+  (junction (at 199.39 114.935) (diameter 0) (color 0 0 0 0)
+  )
   (junction (at 199.39 92.71) (diameter 0) (color 0 0 0 0)
   )
@@
     (stroke (width 0) (type default) (color 0 0 0 0))
   )
-  (wire (pts (xy 186.69 109.855) (xy 199.39 109.855))
-    (stroke (width 0) (type default) (color 0 0 0 0))
-  )
-  (wire (pts (xy 199.39 107.95) (xy 199.39 109.855))
-    (stroke (width 0) (type default) (color 0 0 0 0))
-  )
   (wire (pts (xy 187.325 67.945) (xy 199.39 67.945))
     (stroke (width 0) (type default) (color 0 0 0 0))
   )
+  (wire (pts (xy 176.53 114.935) (xy 199.39 114.935))
+    (stroke (width 0) (type default) (color 0 0 0 0))
+  )
   (wire (pts (xy 187.96 100.965) (xy 199.39 100.965))
     (stroke (width 0) (type default) (color 0 0 0 0))
@@
     (stroke (width 0) (type default) (color 0 0 0 0))
   )
+  (wire (pts (xy 172.72 103.505) (xy 172.72 109.855))
+    (stroke (width 0) (type default) (color 0 0 0 0))
+  )
   (polyline (pts (xy 160.02 56.515) (xy 220.345 56.515))
     (stroke (width 0) (type default) (color 0 0 0 0))
@@
     (stroke (width 0) (type default) (color 0 0 0 0))
   )
+  (wire (pts (xy 172.72 120.015) (xy 172.72 121.285))
+    (stroke (width 0) (type default) (color 0 0 0 0))
+  )
   (wire (pts (xy 166.37 67.945) (xy 179.705 67.945))
     (stroke (width 0) (type default) (color 0 0 0 0))
@@
     (stroke (width 0) (type default) (color 0 0 0 0))
   )
-  (wire (pts (xy 199.39 109.855) (xy 214.63 109.855))
-    (stroke (width 0) (type default) (color 0 0 0 0))
-  )
   (wire (pts (xy 199.39 67.945) (xy 214.63 67.945))
     (stroke (width 0) (type default) (color 0 0 0 0))
   )
-  (polyline (pts (xy 160.02 56.515) (xy 160.02 120.65))
+  (polyline (pts (xy 160.02 56.515) (xy 160.02 127))
     (stroke (width 0) (type default) (color 0 0 0 0))
   )
@@
     (stroke (width 0) (type default) (color 0 0 0 0))
   )
-  (polyline (pts (xy 220.345 120.65) (xy 220.345 56.515))
+  (polyline (pts (xy 219.71 127) (xy 220.345 56.515))
     (stroke (width 0) (type default) (color 0 0 0 0))
   )
@@
     (stroke (width 0) (type default) (color 0 0 0 0))
   )
+  (wire (pts (xy 199.39 113.03) (xy 199.39 114.935))
+    (stroke (width 0) (type default) (color 0 0 0 0))
+  )
   (wire (pts (xy 187.325 92.71) (xy 199.39 92.71))
     (stroke (width 0) (type default) (color 0 0 0 0))
@@
     (stroke (width 0) (type default) (color 0 0 0 0))
   )
-  (polyline (pts (xy 160.02 120.65) (xy 220.345 120.65))
+  (polyline (pts (xy 160.02 127) (xy 219.71 127))
+    (stroke (width 0) (type default) (color 0 0 0 0))
+  )
+  (wire (pts (xy 199.39 114.935) (xy 214.63 114.935))
     (stroke (width 0) (type default) (color 0 0 0 0))
   )
@@
     (stroke (width 0) (type default) (color 0 0 0 0))
   )
-  (wire (pts (xy 172.72 109.855) (xy 172.72 111.76))
-    (stroke (width 0) (type default) (color 0 0 0 0))
-  )
-  (wire (pts (xy 172.72 109.855) (xy 179.07 109.855))
-    (stroke (width 0) (type default) (color 0 0 0 0))
-  )
   (wire (pts (xy 88.9 83.82) (xy 94.615 83.82))
     (stroke (width 0) (type default) (color 0 0 0 0))
@@
   (wire (pts (xy 129.54 85.725) (xy 129.54 83.82))
     (stroke (width 0) (type default) (color 0 0 0 0))
+  )
+  (text "PS should be tied to ground for SPI" (at 180.34 117.475 0)
+    (effects (font (size 1 1)) (justify left bottom))
   )
   (text "DEBUG" (at 160.02 55.88 0)
     (effects (font (size 1.27 1.27)) (justify left bottom))
   )
-  (text "Tie PS to ground for SPI" (at 184.785 113.03 0)
-    (effects (font (size 1 1)) (justify left bottom))
-  )
   (text "MS5611" (at 90.805 67.31 180)
     (effects (font (size 1.27 1.27)) (justify right bottom))
@@
     (effects (font (size 1.27 1.27)) (justify right bottom))
   )
+  (label "PS" (at 214.63 114.935 180)
+    (effects (font (size 1.27 1.27)) (justify right bottom))
+  )
   (label "+3V3" (at 214.63 67.945 180)
     (effects (font (size 1.27 1.27)) (justify right bottom))
@@
     (effects (font (size 1.27 1.27)) (justify right bottom))
   )
+  (label "+3V3" (at 172.72 103.505 270)
+    (effects (font (size 1.27 1.27)) (justify right bottom))
+  )
   (label "+3V3" (at 132.715 71.12 270)
     (effects (font (size 1.27 1.27)) (justify right bottom))
@@
     (effects (font (size 1.27 1.27)) (justify left bottom))
   )
-  (label "PS" (at 214.63 109.855 180)
-    (effects (font (size 1.27 1.27)) (justify right bottom))
-  )
   (hierarchical_label "MISO" (shape output) (at 172.72 76.2 180)
     (effects (font (size 1.27 1.27)) (justify right))
@@
     )
     (property "Datasheet" "https://www.te.com/commerce/DocumentDelivery/DDEController?Action=srchrtrv&DocNm=MS5611-01BA03&DocType=Data+Sheet&DocLang=English" (id 3) (at 104.775 88.9 0)
+      (effects (font (size 1.27 1.27)) hide)
+    )
+    (property "Digikey" "https://www.digikey.com/en/products/detail/te-connectivity-measurement-specialties/MS561101BA03-50/5277445" (id 4) (at 104.775 88.9 0)
       (effects (font (size 1.27 1.27)) hide)
     )
@@
     (pin "2")
   )
+  (symbol (lib_id "power:GND") (at 172.72 121.285 0) (unit 1)
+    (in_bom yes) (on_board yes)
+    (property "Reference" "#PWR0113" (id 0) (at 172.72 127.635 0)
+      (effects (font (size 1.27 1.27)) hide)
+    )
+    (property "Value" "GND" (id 1) (at 168.91 122.555 0))
+    (property "Footprint" "" (id 2) (at 172.72 121.285 0)
+      (effects (font (size 1.27 1.27)) hide)
+    )
+    (property "Datasheet" "" (id 3) (at 172.72 121.285 0)
+      (effects (font (size 1.27 1.27)) hide)
+    )
+    (pin "1")
+  )
   (symbol (lib_id "Device:C_Small") (at 129.54 81.28 0) (unit 1)
     (in_bom yes) (on_board yes) (fields_autoplaced)
@@
     (pin "1")
   )
-  (symbol (lib_id "power:GND") (at 172.72 111.76 0) (unit 1)
-    (in_bom yes) (on_board yes) (fields_autoplaced)
-    (property "Reference" "#PWR0113" (id 0) (at 172.72 118.11 0)
-      (effects (font (size 1.27 1.27)) hide)
-    )
-    (property "Value" "GND" (id 1) (at 172.72 116.84 0))
-    (property "Footprint" "" (id 2) (at 172.72 111.76 0)
-      (effects (font (size 1.27 1.27)) hide)
-    )
-    (property "Datasheet" "" (id 3) (at 172.72 111.76 0)
-      (effects (font (size 1.27 1.27)) hide)
-    )
-    (pin "1")
-  )
   (symbol (lib_id "Connector:TestPoint") (at 199.39 99.695 0) (unit 1)
     (in_bom yes) (on_board yes)
@@
     )
     (property "Datasheet" "~" (id 3) (at 204.47 99.695 0)
+      (effects (font (size 1.27 1.27)) hide)
+    )
+    (pin "1")
+  )
+  (symbol (lib_id "Connector:TestPoint") (at 199.39 113.03 0) (unit 1)
+    (in_bom yes) (on_board yes)
+    (property "Reference" "TP18" (id 0) (at 200.66 109.22 0)
+      (effects (font (size 1.27 1.27)) (justify left))
+    )
+    (property "Value" "Header" (id 1) (at 200.66 111.76 0)
+      (effects (font (size 1.27 1.27)) (justify left))
+    )
+    (property "Footprint" "Connector_PinHeader_2.54mm:PinHeader_1x01_P2.54mm_Vertical" (id 2) (at 204.47 113.03 0)
+      (effects (font (size 1.27 1.27)) hide)
+    )
+    (property "Datasheet" "~" (id 3) (at 204.47 113.03 0)
       (effects (font (size 1.27 1.27)) hide)
     )
@@
     (pin "1")
   )
-  (symbol (lib_id "Connector:TestPoint") (at 199.39 107.95 0) (unit 1)
-    (in_bom yes) (on_board yes)
-    (property "Reference" "TP18" (id 0) (at 200.66 104.14 0)
-      (effects (font (size 1.27 1.27)) (justify left))
-    )
-    (property "Value" "Header" (id 1) (at 200.66 106.68 0)
-      (effects (font (size 1.27 1.27)) (justify left))
-    )
-    (property "Footprint" "Connector_PinHeader_2.54mm:PinHeader_1x01_P2.54mm_Vertical" (id 2) (at 204.47 107.95 0)
-      (effects (font (size 1.27 1.27)) hide)
-    )
-    (property "Datasheet" "~" (id 3) (at 204.47 107.95 0)
-      (effects (font (size 1.27 1.27)) hide)
-    )
-    (pin "1")
+  (symbol (lib_id "Jumper:SolderJumper_3_Open") (at 172.72 114.935 90) (unit 1)
+    (in_bom yes) (on_board yes) (fields_autoplaced)
+    (property "Reference" "JP20" (id 0) (at 171.069 115.3688 90)
+      (effects (font (size 1.27 1.27)) (justify left))
+    )
+    (property "Value" "SolderJumper_3_Open" (id 1) (at 170.6681 114.935 0)
+      (effects (font (size 1.27 1.27)) hide)
+    )
+    (property "Footprint" "Jumper:SolderJumper-3_P1.3mm_Open_RoundedPad1.0x1.5mm" (id 2) (at 172.72 114.935 0)
+      (effects (font (size 1.27 1.27)) hide)
+    )
+    (property "Datasheet" "~" (id 3) (at 172.72 114.935 0)
+      (effects (font (size 1.27 1.27)) hide)
+    )
+    (pin "1")
+    (pin "2")
+    (pin "3")
   )
   (symbol (lib_id "Device:C_Small") (at 119.38 81.28 0) (unit 1)
@@
     (pin "1")
   )
-  (symbol (lib_id "Device:R") (at 182.88 109.855 90) (unit 1)
-    (in_bom yes) (on_board yes)
-    (property "Reference" "R3" (id 0) (at 182.88 107.315 90))
-    (property "Value" "10K" (id 1) (at 182.88 109.855 90))
-    (property "Footprint" "" (id 2) (at 182.88 111.633 90)
-      (effects (font (size 1.27 1.27)) hide)
-    )
-    (property "Datasheet" "~" (id 3) (at 182.88 109.855 0)
-      (effects (font (size 1.27 1.27)) hide)
-    )
-    (pin "1")
-    (pin "2")
-  )
 )
