File: hardware/dev-board/kicad/hierarchical_sheets/sx1262.kicad_sch (KiCad schematic)
At the start: 0 parts

Commit message: rf is hard
Parts:
- added C?: 10pF, symbol Device:C
- added C?: 0.47μF, symbol Device:C
- added C?: 0.1μF, symbol Device:C
- added FB?: 2506036017H0, Capacitor_SMD:C_0603_1608Metric_Pad1.08x0.95mm_HandSolder, symbol Device:FerriteBead
- added L?: LPS3010-153, symbol Device:L
- added R?: 220Ω, symbol Device:R
- added U?: sx1262, symbol SRAD-FC:sx1262
- added X?: ECS-TXO-25CSMV-320-BM-TR, SRAD-FC:ECS-TXO-25CSMV-320-BM-TR, symbol SRAD-FC:ECS-TXO-25CSMV-320-BM-TR
Connections:
- new net: C?.2, R?.1
- new net: C?.1, X?.3 (OUT)
- new net: C?.1, FB?.2, X?.4 (Vcc)
- new net DCC_SW: L?.2, U?.9 (DCC_SW)
- new net DIO3: FB?.1, U?.6 (DIO3)
- new net GND: C?.2, C?.2, U?.0 (GND), U?.2 (GND), U?.20 (GND), U?.5 (GND), U?.8 (GND), X?.1 (NC), X?.2 (GND)
- new net MISO: U?.16 (MISO)
- new net MOSI: U?.17 (MOSI)
- new net SCK: U?.18 (SCK)
- new net VREG: C?.1, L?.1, U?.7 (VREG)
- new net XTA: R?.2, U?.3 (XTA)
- new net XTB: U?.4 (XTB)
- new net ~{CS}: U?.19 (~{CS})
- no-connect marks 0 -> 1
Other:
- company: (none) -> Missouri S&T Rocket Design Team

Commit message: update
Parts:
- added C? (x3): 0.1μF, symbol Device:C_Small
- added C? (x2): 10nF, symbol Device:C_Small
- added JP? (x7): SolderJumper_2_Open, Jumper:SolderJumper-2_P1.3mm_Open_RoundedPad1.0x1.5mm, symbol Jumper:SolderJumper_2_Open
- added JP?: SolderJumper_3_Open, Jumper:SolderJumper-3_P1.3mm_Open_RoundedPad1.0x1.5mm, symbol Jumper:SolderJumper_3_Open
- added R?: 10K, symbol Device:R_Small
- added TP? (x14): Header, Connector_PinHeader_2.54mm:PinHeader_1x01_P2.54mm_Vertical, symbol Connector:TestPoint
- added U?: pe4242, symbol SRAD-FC:pe4242
- U?: footprint (none) -> Package_DFN_QFN:QFN-24-1EP_4x4mm_P0.5mm_EP2.6x2.6mm_ThermalVias; Digikey (none) -> https://www.digikey.com/en/products/detail/semtech-corporat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
Connections:
- net GND: now also C?.2, C?.2, C?.2, C?.2, C?.2, JP?.1 (A)
- net MISO: now also JP?.1 (A), JP?.2 (B), TP?.1
- net MOSI: now also JP?.1 (A), JP?.2 (B), TP?.1
- net SCK: now also JP?.1 (A), JP?.2 (B), TP?.1
- net ~{CS}: now also JP?.1 (A), JP?.2 (B), TP?.1
- net VCC_RADIO: now reaches U?.1 (VDD_IN)
- net VCC_RADIO: now also U?.10 (VBAT), U?.11 (VBAT_IO), C?.1, C?.1, C?.1, C?.1, R?.1
- net DIO2: now reaches U?.12 (DIO2)
- net INT: now reaches U?.13 (DIO1)
- net INT: now also JP?.1 (A), JP?.2 (B), TP?.1
- net BUSY: now reaches U?.14 (BUSY)
- net BUSY: now also JP?.1 (A), JP?.2 (B), TP?.1
- net ~{NRESET}: now reaches U?.15 (~{NRESET})
- net ~{NRESET}: now also C?.1, R?.2
- net TCXO_VCC: now reaches C?.1, FB?.2, X?.4 (Vcc)
- net TCXO_VCC: now also TP?.1
- new net +3V3: JP?.1 (A), JP?.2 (B), TP?.1
- new net D_SEL: JP?.2 (C), TP?.1
- new net GPS_VCC: JP?.3 (B), TP?.1
- new net PIO15: TP?.1
- new net V_BCKP: TP?.1
- new net ~{RESET}: TP?.1
- new net ~{SAFEBOOT}: TP?.1
Other:
- note added: "*Remove for final*"
- note added: "BUSY low = chip ready for command"
- note added: "DEBUG"
- note added: "D_SEL should be tied to ground for SPI"
- note added: "TCXO for temperature stability"
- note added: "~{RESET} is active low"
- note added: "~{SAFEBOOT} is active low, internal pullup"
- moved on the sheet: C?, FB?, L?, R?, U?, X?

Commit message: some rf work
Parts:
- U?: footprint (none) -> Package_TO_SOT_SMD:SOT-363_SC-70-6; Digikey (none) -> https://www.digikey.com/en/products/detail/psemi/PE42421SCA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
Changed lines of the file:
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@@
     (property "Reference" "U?" (id 0) (at 179.3875 107.95 0))
     (property "Value" "pe4242" (id 1) (at 179.3875 110.49 0))
-    (property "Footprint" "" (id 2) (at 156.21 114.3 0)
+    (property "Footprint" "Package_TO_SOT_SMD:SOT-363_SC-70-6" (id 2) (at 156.21 114.3 0)
       (effects (font (size 1.27 1.27)) hide)
     )
-    (property "Datasheet" "" (id 3) (at 156.21 114.3 0)
+    (property "Datasheet" "https://www.psemi.com/pdf/datasheets/pe42421ds.pdf" (id 3) (at 156.21 114.3 0)
       (effects (font (size 1.27 1.27)) hide)
     )
+    (property "Digikey" "https://www.digikey.com/en/products/detail/psemi/PE42421SCAA-Z/3728588" (id 4) (at 179.07 120.015 0)
+      (effects (font (size 1.27 1.27)) hide)
+    )
