File: hardware/kicad/hierarchical_sheets/mb85rs2mtapnf.kicad_sch (KiCad schematic)
At the start: 0 parts

Commit message: FRAM schematic
Parts:
- added U5: MB85RS2, symbol Memory_NVRAM:MB85RS16
Changed lines of the file:
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@@
     (company "Missouri S&T Rocket Design Team")
   )
+  (symbol (lib_id "Memory_NVRAM:MB85RS16") (at 168.91 96.52 0) (unit 1)
+    (in_bom yes) (on_board yes) (dnp no) (fields_autoplaced)
+    (property "Reference" "U5" (at 171.1041 86.36 0)
+      (effects (font (size 1.27 1.27)) (justify left))
+    )
+    (property "Value" "MB85RS2" (at 171.1041 88.9 0)
+      (effects (font (size 1.27 1.27)) (justify left))
+    )
+    (property "Footprint" "" (at 160.02 97.79 0)
+      (effects (font (size 1.27 1.27)) hide)
+    )
+    (property "Datasheet" "http://www.fujitsu.com/downloads/MICRO/fsa/pdf/products/memory/fram/MB85RS16-DS501-00014-6v0-E.pdf" (at 160.02 97.79 0)
+      (effects (font (size 1.27 1.27)) hide)
+    )
+    (pin "1")
+    (pin "2")
+    (pin "3")
+    (pin "4")
+    (pin "5")
+    (pin "6")
+    (pin "7")
+    (pin "8")
+    (instances
+      (project "FC"
+        (path "/54cce219-8b98-4e71-96c4-f9ee784aa3bc/ec693876-f9f5-4d00-b73f-be61605a2d0a"
+          (reference "U5") (unit 1)
+        )
+      )
+    )
+  )
 )
