File: hardware/kicad/hierarchical_sheets/mb85rs2mtapnf.kicad_sch (KiCad schematic)
At the start: 3 parts, among them U10 MB85RS2

Commit message: Storage Update
Made changes following Seth's advice
Parts:
- R18: value 1k -> 10k
- U10: footprint (none) -> Package_SO:SOIC-8_3.9x4.9mm_P1.27mm
Connections:
- net +3.3V: now also R18.2
- net ~{CS}: now also R18.1, U10.1 (~{CS}); no longer R18.2
Other:
- moved on the sheet: R18
Changed lines of the file:
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@@
   (junction (at 49.53 27.94) (diameter 0) (color 0 0 0 0)
   )
+  (junction (at 34.29 43.18) (diameter 0) (color 0 0 0 0)
+  )
   (junction (at 49.53 55.88) (diameter 0) (color 0 0 0 0)
   )
   (no_connect (at 39.37 38.1))
-  (wire (pts (xy 34.29 50.8) (xy 35.56 50.8))
-    (stroke (width 0) (type default))
-  )
   (wire (pts (xy 49.53 27.94) (xy 49.53 33.02))
     (stroke (width 0) (type default))
@@
     (stroke (width 0) (type default))
   )
+  (wire (pts (xy 29.21 50.8) (xy 34.29 50.8))
+    (stroke (width 0) (type default))
+  )
+  (wire (pts (xy 30.48 43.18) (xy 34.29 43.18))
+    (stroke (width 0) (type default))
+  )
   (wire (pts (xy 71.12 38.1) (xy 59.69 38.1))
     (stroke (width 0) (type default))
   )
+  (wire (pts (xy 34.29 43.18) (xy 39.37 43.18))
+    (stroke (width 0) (type default))
+  )
   (wire (pts (xy 85.09 55.88) (xy 49.53 55.88))
     (stroke (width 0) (type default))
@@
   )
   (wire (pts (xy 85.09 27.94) (xy 49.53 27.94))
-    (stroke (width 0) (type default))
-  )
-  (wire (pts (xy 35.56 43.18) (xy 39.37 43.18))
     (stroke (width 0) (type default))
   )
@@
     (effects (font (size 1.27 1.27)) (justify right))
   )
-  (hierarchical_label "~{CS}" (shape input) (at 34.29 50.8 180) (fields_autoplaced)
+  (hierarchical_label "~{CS}" (shape input) (at 30.48 43.18 180) (fields_autoplaced)
     (effects (font (size 1.27 1.27)) (justify right))
   )
@@
     (effects (font (size 1.27 1.27)) (justify left))
   )
-  (symbol (lib_id "Device:R") (at 35.56 46.99 0) (unit 1)
+  (symbol (lib_id "power:+3.3V") (at 29.21 50.8 0) (unit 1)
+    (in_bom yes) (on_board yes) (dnp no)
+    (property "Reference" "#PWR062" (at 29.21 54.61 0)
+      (effects (font (size 1.27 1.27)) hide)
+    )
+    (property "Value" "+3.3V" (at 29.21 46.99 0)
+      (effects (font (size 1.27 1.27)))
+    )
+    (property "Footprint" "" (at 29.21 50.8 0)
+      (effects (font (size 1.27 1.27)) hide)
+    )
+    (property "Datasheet" "" (at 29.21 50.8 0)
+      (effects (font (size 1.27 1.27)) hide)
+    )
+    (pin "1")
+    (instances
+      (project "FC"
+        (path "/54cce219-8b98-4e71-96c4-f9ee784aa3bc/ec693876-f9f5-4d00-b73f-be61605a2d0a"
+          (reference "#PWR062") (unit 1)
+        )
+      )
+    )
+  )
+  (symbol (lib_id "Device:R") (at 34.29 46.99 0) (unit 1)
     (in_bom yes) (on_board yes) (dnp no) (fields_autoplaced)
-    (property "Reference" "R18" (at 38.1 45.72 0)
+    (property "Reference" "R18" (at 36.83 45.72 0)
       (effects (font (size 1.27 1.27)) (justify left))
     )
-    (property "Value" "1k" (at 38.1 48.26 0)
+    (property "Value" "10k" (at 36.83 48.26 0)
       (effects (font (size 1.27 1.27)) (justify left))
     )
-    (property "Footprint" "Resistor_SMD:R_0603_1608Metric" (at 33.782 46.99 90)
-      (effects (font (size 1.27 1.27)) hide)
-    )
-    (property "Datasheet" "~" (at 35.56 46.99 0)
+    (property "Footprint" "Resistor_SMD:R_0603_1608Metric" (at 32.512 46.99 90)
+      (effects (font (size 1.27 1.27)) hide)
+    )
+    (property "Datasheet" "~" (at 34.29 46.99 0)
       (effects (font (size 1.27 1.27)) hide)
     )
@@
       (effects (font (size 1.27 1.27)) (justify left))
     )
-    (property "Footprint" "" (at 40.64 41.91 0)
+    (property "Footprint" "Package_SO:SOIC-8_3.9x4.9mm_P1.27mm" (at 40.64 41.91 0)
       (effects (font (size 1.27 1.27)) hide)
     )
@@
       (effects (font (size 1.27 1.27)) hide)
     )
-    (property "Digikey" "https://www.digikey.com/en/products/detail/kaga-fei-america-inc/MB85RS2MTAPNF-G-BDERE1/7604211" (at 49.53 40.64 0)
-      (effects (font (size 1.27 1.27)) hide)
-    )
+    (property "Digikey" "https://www.digikey.com/en/products/detail/kaga-fei-america-inc/MB85RS2MTAPNF-G-BDERE1/7604211" (at 49.53 30.48 0)
+      (effects (font (size 1.27 1.27)) hide)
+    )

Commit message: making formatting more consistent
Other:
- note removed: "Comments: - The ~{CS} Pullup resistor should be between the ~{CS} and 3.3V, not in series between the chip and the microcontroller. Also, make the ~{CS} Resistor 10k. The only purpose of this resistor is to ensure that the chip stays inactive while the microcontroller is being initially programmed since during programming the chip will be unable to hold the various ~{CS} lines high. A higher valu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"
- moved on the sheet: C15, R18, U10

Commit message: formatting
Parts:
- renumbered U10 to U11
Changed lines of the file:
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@@
   (symbol (lib_id "power:+3.3V") (at 102.87 97.155 0) (unit 1)
     (in_bom yes) (on_board yes) (dnp no)
-    (property "Reference" "#PWR062" (at 102.87 100.965 0)
+    (property "Reference" "#PWR042" (at 102.87 100.965 0)
       (effects (font (size 1.27 1.27)) hide)
     )
@@
       (project "FC"
         (path "/54cce219-8b98-4e71-96c4-f9ee784aa3bc/ec693876-f9f5-4d00-b73f-be61605a2d0a"
-          (reference "#PWR062") (unit 1)
+          (reference "#PWR042") (unit 1)
         )
       )
@@
   (symbol (lib_id "power:GND") (at 123.19 103.505 0) (unit 1)
     (in_bom yes) (on_board yes) (dnp no) (fields_autoplaced)
-    (property "Reference" "#PWR043" (at 123.19 109.855 0)
+    (property "Reference" "#PWR044" (at 123.19 109.855 0)
       (effects (font (size 1.27 1.27)) hide)
     )
@@
       (project "FC"
         (path "/54cce219-8b98-4e71-96c4-f9ee784aa3bc/ec693876-f9f5-4d00-b73f-be61605a2d0a"
-          (reference "#PWR043") (unit 1)
+          (reference "#PWR044") (unit 1)
         )
       )
@@
   (symbol (lib_id "power:+3.3V") (at 123.19 73.025 0) (unit 1)
     (in_bom yes) (on_board yes) (dnp no)
-    (property "Reference" "#PWR042" (at 123.19 76.835 0)
+    (property "Reference" "#PWR043" (at 123.19 76.835 0)
       (effects (font (size 1.27 1.27)) hide)
     )
@@
       (project "FC"
         (path "/54cce219-8b98-4e71-96c4-f9ee784aa3bc/ec693876-f9f5-4d00-b73f-be61605a2d0a"
-          (reference "#PWR042") (unit 1)
+          (reference "#PWR043") (unit 1)
         )
       )
@@
   (symbol (lib_id "Memory_NVRAM:MB85RS16") (at 123.19 86.995 0) (unit 1)
     (in_bom yes) (on_board yes) (dnp no) (fields_autoplaced)
-    (property "Reference" "U10" (at 125.3841 76.835 0)
+    (property "Reference" "U11" (at 125.3841 76.835 0)
       (effects (font (size 1.27 1.27)) (justify left))
     )
@@
       (project "FC"
         (path "/54cce219-8b98-4e71-96c4-f9ee784aa3bc/ec693876-f9f5-4d00-b73f-be61605a2d0a"
-          (reference "U10") (unit 1)
+          (reference "U11") (unit 1)
         )
       )
