File: hardware/kicad/hierarchical_sheets/mb85rs2mtapnf.kicad_sch (KiCad schematic)
At the start: 3 parts, among them U11 MB85RS2

Commit message: formatting / exported pdf
Other:
- title: SRAD-FC -> Storage (MB85RS2)
Changed lines of the file:
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@@
   (paper "USLetter")
   (title_block
-    (title "SRAD-FC")
+    (title "Storage (MB85RS2)")
     (company "Missouri S&T Rocket Design Team")
     (comment 1 "Cliffford Matteson")
