File: hardware/kicad/hierarchical_sheets/bmi-270.kicad_sch (KiCad schematic)
At the start: 0 parts

Commit message: created microcontroller schematic
Other:
- company: (none) -> Missouri S&T Rocket Design Team
- title: (none) -> SRAD-FC
Changed lines of the file:
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@@
 (kicad_sch (version 20230121) (generator eeschema)
-  (paper "A4")
+  (paper "USLetter")
+  (title_block
+    (title "SRAD-FC")
+    (company "Missouri S&T Rocket Design Team")
+  )
 )

Commit message: Added Resistor
Parts:
- added R2: R, symbol Device:R
Changed lines of the file:
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@@
     (company "Missouri S&T Rocket Design Team")
   )
+  (symbol (lib_id "Device:R") (at 133.35 66.04 0) (unit 1)
+    (in_bom yes) (on_board yes) (dnp no) (fields_autoplaced)
+    (property "Reference" "R2" (at 135.89 64.77 0)
+      (effects (font (size 1.27 1.27)) (justify left))
+    )
+    (property "Value" "R" (at 135.89 67.31 0)
+      (effects (font (size 1.27 1.27)) (justify left))
+    )
+    (property "Footprint" "" (at 131.572 66.04 90)
+      (effects (font (size 1.27 1.27)) hide)
+    )
+    (property "Datasheet" "~" (at 133.35 66.04 0)
+      (effects (font (size 1.27 1.27)) hide)
+    )
+    (pin "1")
+    (pin "2")
+    (instances
+      (project "FC"
+        (path "/54cce219-8b98-4e71-96c4-f9ee784aa3bc/7e43dc21-d4ed-4dfe-b96f-060fb7f0f8ce"
+          (reference "R2") (unit 1)
+        )
+      )
+    )
+  )
 )
