File: hardware/kicad/hierarchical_sheets/bmi-270.kicad_sch (KiCad schematic)
At the start: 1 part, among them U8 BMI270

Commit message: Fixed schematic file
Parts:
- removed U8: BMI270, BMI270:XDCR_BMI270, symbol BMI270:BMI270
- added BMI270_4WireSPI: BMI270, BMI270:XDCR_BMI270, symbol BMI270:BMI270
- added C6, C7: 100nF, symbol Device:C_Small
Connections:
- new net CSB: BMI270_4WireSPI.12 (CSB)
- new net GNDD: BMI270_4WireSPI.6 (GNDIO), BMI270_4WireSPI.7 (GND), C6.1, C7.1
- new net INT1: BMI270_4WireSPI.4 (INT1)
- new net INT2: BMI270_4WireSPI.9 (INT2)
- new net SCK: BMI270_4WireSPI.13 (SCx)
- new net SDI/MOSI: BMI270_4WireSPI.14 (SDx)
- new net SDO/MISO: BMI270_4WireSPI.1 (SDO)
- new net VDD: BMI270_4WireSPI.8 (VDD), C6.2
- new net VDDIO: BMI270_4WireSPI.5 (VDDIO), C7.2

Commit message: Added Schematic stuff
Parts:
- removed C6, C7: 100nF, symbol Device:C_Small
- added 100nF, 100nF1: C_Small, symbol Device:C_Small
Connections:
- net VDDIO is gone; now on net +3.3V: BMI270_4WireSPI.5 (VDDIO)
- net CSB renamed ~{CS}
- net GNDD renamed GND
- net GND: now also 100nF.2, 100nF1.2
- net INT1: no longer names the net of BMI270_4WireSPI.4 (INT1)
- net INT2: no longer names the net of BMI270_4WireSPI.9 (INT2)
- net SDI/MOSI renamed MOSI
- net SDO/MISO renamed MISO
- net VDD renamed +3.3V
- net +3.3V: now also 100nF.1, 100nF1.1
- no-connect marks 0 -> 2
Other:
- note added: "Max Current: 0.97mA"

Commit message: Finnished Schematic?
Parts:
- added R23: 10K, symbol Device:R
- renumbered 100nF to 100n, 100nF1 to 100n
Connections:
- net +3.3V: now also 100n.2, 100n.2, R23.2; no longer 100n.1, 100n.1
- net GND: now also 100n.1, 100n.1; no longer 100n.2, 100n.2
- net ~{CS}: now also R23.1
- no-connect marks 2 -> 6
Other:
- moved on the sheet: 100n

Commit message: started linking together FC, changed cs directions
Changed lines of the file:
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@@
     (effects (font (size 1.27 1.27)) (justify right))
   )
-  (hierarchical_label "~{CS}" (shape output) (at 99.06 104.14 180) (fields_autoplaced)
+  (hierarchical_label "~{CS}" (shape input) (at 99.06 104.14 180) (fields_autoplaced)
     (effects (font (size 1.27 1.27)) (justify right))
   )

Commit message: added imu interrupt
Connections:
- net INT: now reaches BMI270_4WireSPI.4 (INT1)
- no-connect marks 6 -> 5
Other:
- moved on the sheet: R23
Changed lines of the file:
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@@
     (company "Missouri S&T Rocket Design Team")
   )
+  (junction (at 101.6 104.14) (diameter 0) (color 0 0 0 0)
+  )
   (junction (at 129.54 87.63) (diameter 0) (color 0 0 0 0)
   )
@@
   )
   (junction (at 111.76 74.93) (diameter 0) (color 0 0 0 0)
-  )
-  (junction (at 107.95 104.14) (diameter 0) (color 0 0 0 0)
   )
   (junction (at 121.92 83.82) (diameter 0) (color 0 0 0 0)
@@
   (no_connect (at 119.38 109.22))
   (no_connect (at 142.24 104.14))
-  (no_connect (at 119.38 106.68))
   (no_connect (at 142.24 101.6))
   (wire (pts (xy 132.08 119.38) (xy 129.54 119.38))
@@
     (stroke (width 0) (type default))
   )
-  (wire (pts (xy 107.95 119.38) (xy 85.09 119.38))
+  (wire (pts (xy 101.6 127) (xy 78.74 127))
     (stroke (width 0) (type default))
   )
@@
     (stroke (width 0) (type default))
   )
-  (wire (pts (xy 107.95 113.03) (xy 107.95 119.38))
+  (wire (pts (xy 101.6 120.65) (xy 101.6 127))
     (stroke (width 0) (type default))
   )
@@
     (stroke (width 0) (type default))
   )
-  (wire (pts (xy 107.95 105.41) (xy 107.95 104.14))
+  (wire (pts (xy 101.6 104.14) (xy 101.6 113.03))
     (stroke (width 0) (type default))
   )
@@
     (stroke (width 0) (type default))
   )
-  (wire (pts (xy 99.06 104.14) (xy 107.95 104.14))
+  (wire (pts (xy 99.06 104.14) (xy 101.6 104.14))
     (stroke (width 0) (type default))
   )
@@
     (stroke (width 0) (type default))
   )
+  (wire (pts (xy 111.76 106.68) (xy 119.38 106.68))
+    (stroke (width 0) (type default))
+  )
   (wire (pts (xy 99.06 99.06) (xy 119.38 99.06))
     (stroke (width 0) (type default))
   )
-  (wire (pts (xy 85.09 115.57) (xy 85.09 119.38))
+  (wire (pts (xy 78.74 123.19) (xy 78.74 127))
     (stroke (width 0) (type default))
   )
@@
     (stroke (width 0) (type default))
   )
-  (wire (pts (xy 107.95 104.14) (xy 119.38 104.14))
+  (wire (pts (xy 101.6 104.14) (xy 119.38 104.14))
     (stroke (width 0) (type default))
   )
@@
     (at 162.56 160.02 0)
     (effects (font (size 2 2) (thickness 0.4) bold (color 255 48 0 1)) (justify left bottom))
+  )
+  (hierarchical_label "INT" (shape output) (at 111.76 106.68 180) (fields_autoplaced)
+    (effects (font (size 1.27 1.27)) (justify right))
   )
   (hierarchical_label "MOSI" (shape output) (at 99.06 99.06 180) (fields_autoplaced)
@@
     )
   )
-  (symbol (lib_id "power:+3.3V") (at 85.09 115.57 0) (unit 1)
-    (in_bom yes) (on_board yes) (dnp no) (fields_autoplaced)
-    (property "Reference" "#PWR041" (at 85.09 119.38 0)
-      (effects (font (size 1.27 1.27)) hide)
-    )
-    (property "Value" "+3.3V" (at 85.09 110.49 0)
+  (symbol (lib_id "power:+3.3V") (at 78.74 123.19 0) (unit 1)
+    (in_bom yes) (on_board yes) (dnp no) (fields_autoplaced)
+    (property "Reference" "#PWR041" (at 78.74 127 0)
+      (effects (font (size 1.27 1.27)) hide)
+    )
+    (property "Value" "+3.3V" (at 78.74 118.11 0)
       (effects (font (size 1.27 1.27)))
     )
-    (property "Footprint" "" (at 85.09 115.57 0)
-      (effects (font (size 1.27 1.27)) hide)
-    )
-    (property "Datasheet" "" (at 85.09 115.57 0)
+    (property "Footprint" "" (at 78.74 123.19 0)
+      (effects (font (size 1.27 1.27)) hide)
+    )
+    (property "Datasheet" "" (at 78.74 123.19 0)
       (effects (font (size 1.27 1.27)) hide)
     )
@@
     )
   )
-  (symbol (lib_id "Device:R") (at 107.95 109.22 0) (unit 1)
-    (in_bom yes) (on_board yes) (dnp no) (fields_autoplaced)
-    (property "Reference" "R23" (at 110.49 107.95 0)
+  (symbol (lib_id "Device:R") (at 101.6 116.84 0) (unit 1)
+    (in_bom yes) (on_board yes) (dnp no) (fields_autoplaced)
+    (property "Reference" "R23" (at 104.14 115.57 0)
       (effects (font (size 1.27 1.27)) (justify left))
     )
-    (property "Value" "10K" (at 110.49 110.49 0)
+    (property "Value" "10K" (at 104.14 118.11 0)
       (effects (font (size 1.27 1.27)) (justify left))
     )
-    (property "Footprint" "" (at 106.172 109.22 90)
-      (effects (font (size 1.27 1.27)) hide)
-    )
-    (property "Datasheet" "~" (at 107.95 109.22 0)
-      (effects (font (size 1.27 1.27)) hide)
-    )
+    (property "Footprint" "" (at 99.822 116.84 90)
+      (effects (font (size 1.27 1.27)) hide)
+    )
+    (property "Datasheet" "~" (at 101.6 116.84 0)
+      (effects (font (size 1.27 1.27)) hide)
+    )

Commit message: added power and checked schematics
Other:
- note removed: "Comments: - This chip has two supply pins VDDIO and VDD. Both of these pins are 3.3v compatible. Connect them both to 3.3v. Since They are supply pins, place two 100n capacitors between 3.3v and gnd. These are decoupling capacitors for the supply pins and as such they need to be placed near the chip on the PCB. To help us remember this, place them physically close to the supply pins on the schema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"
Changed lines of the file:
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@@
     (effects (font (size 1.27 1.27)) (justify left bottom))
-  )
-  (text "Comments:\n\n- This chip has two supply pins VDDIO and VDD. Both of these pins are 3.3v compatible. Connect them both to 3.3v. Since\n	They are supply pins, place two 100n capacitors between 3.3v and gnd. These are decoupling capacitors for the supply\n	pins and as such they need to be placed near the chip on the PCB. To help us remember this, place them physically\n	close to the supply pins on the schematic. (see microcontroller for example) \n\n- According to pg 123 of the datasheet, the SPI interface (which we are using) is selected by toggling the CSB pin (~{CS})\n	This can be done by the microcontroller. Connect the SPI pins to hierarchical labels as follows:\n		- SDO -> MISO\n		- SDx -> MOSI\n		- SCx -> SCK\n\n- The INT pins can be used as an interrupt whenever certain motion detections occur, we do not really have enough pins to \n	utilize this and so just set INT1 and INT2 as no connect\n\n- Add a ~{CS} pullup resistor between the ~{CS} pin and 3.3v. Make this resistor\n	10k. The only purpose of this resistor is to ensure that the chip stays inactive \n	while the microcontroller is being initially programmed since during programming the chip\n	will be unable to hold the various ~{CS} lines high. (The MOSI/MISO lines \n	are used by the programmer so if this chip starts communicating while\n	the programmer is communicating to the microcontroller it could be really \n	bad.) A higher value resistor is less likely to cause problems during normal \n	operation. \n\n- The OCSB and OSDO pins are used for optical image stabilitization applications. We don't need them so set them as\n	no connection.  \n\n- The ASDx, and ASCx pins are used to allow chaining an i2c sensor to this chip (ex magnetometer). We are just going\n	to connect the magnetometer to the microcontroller so just mark these pins as no connect. \n\n\n			-Seth"
-    (at 162.56 160.02 0)
-    (effects (font (size 2 2) (thickness 0.4) bold (color 255 48 0 1)) (justify left bottom))
   )
   (hierarchical_label "INT" (shape output) (at 111.76 106.68 180) (fields_autoplaced)
