File: hardware/kicad/hierarchical_sheets/ra-01sh.kicad_sch (KiCad schematic)
At the start: 1 part, among them U4 RA-01SH

Commit message: Storage Updated
Didn't save. Added pins to hierarchal sheets. In/Out
Parts:
- removed U4: RA-01SH, RF_Module:RA-01SH, symbol RA-01SH:RA-01SH
Other:
- title: Telemetry Radio (RA-01SH) -> SRAD-FC
Changed lines of the file:
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@@
   (paper "USLetter")
   (title_block
-    (title "Telemetry Radio (RA-01SH)")
-    (date "2023-09-17")
+    (title "SRAD-FC")
     (company "Missouri S&T Rocket Design Team")
-    (comment 1 "Ariel Pilger")
-  )
-  (symbol (lib_id "RA-01SH:RA-01SH") (at 132.08 87.63 0) (unit 1)
-    (in_bom yes) (on_board yes) (dnp no) (fields_autoplaced)
-    (property "Reference" "U4" (at 134.2741 64.77 0)
-      (effects (font (size 1.27 1.27)) (justify left))
-    )
-    (property "Value" "RA-01SH" (at 134.2741 67.31 0)
-      (effects (font (size 1.27 1.27)) (justify left))
-    )
-    (property "Footprint" "RF_Module:RA-01SH" (at 157.48 97.79 0)
-      (effects (font (size 1.27 1.27)) hide)
-    )
-    (property "Datasheet" "https://docs.ai-thinker.com/_media/lora/docs/ra-01sh_specification.pdf" (at 134.2741 69.85 0)
-      (effects (font (size 1.27 1.27)) (justify left))
-    )
-    (property "Digikey" "https://docs.ai-thinker.com/_media/lora/docs/ra-01sh_specification.pdf" (at 134.2741 72.39 0)
-      (effects (font (size 1.27 1.27)) (justify left))
-    )
-    (pin "1")
-    (pin "10")
-    (pin "11")
-    (pin "12")
-    (pin "13")
-    (pin "14")
-    (pin "15")
-    (pin "16")
-    (pin "2")
-    (pin "3")
-    (pin "4")
-    (pin "5")
-    (pin "6")
-    (pin "7")
-    (pin "8")
-    (pin "9")
-    (instances
-      (project "RA-01SH.kicad_sym"
-        (path "/54cce219-8b98-4e71-96c4-f9ee784aa3bc/35031a3a-251a-4009-92bf-5738de5c8c69"
-          (reference "U4") (unit 1)
-        )
-      )
-    )
   )
 )

Commit message: file sync
Parts:
- added J4: CONSMA020.062-G, CONSMA020.062:CONSMA020.062-G, symbol CONSMA020.062-G:CONSMA020.062-G
- added R16: 1K, symbol Device:R
- added U3: RA-01SH, RF_Module:RA-01SH, symbol RA-01SH:RA-01SH
Connections:
- new net: J4.1 (In), U3.1 (ANT)
- new net +3.3V: R16.2, U3.3 (3.3V)
- new net GND: J4.2 (Ext), U3.16 (GND), U3.2 (GND), U3.9 (GND)
- new net MISO: U3.13 (MISO)
- new net MOSI: U3.14 (MOSI)
- new net SCK: U3.12 (SCK)
- new net ~{CS}: R16.1, U3.15 (~{NSS})
- no-connect marks 0 -> 3
Other:
- title: SRAD-FC -> Telemetry Radio (RA-01SH)
Changed lines of the file:
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@@
   (paper "USLetter")
   (title_block
-    (title "SRAD-FC")
+    (title "Telemetry Radio (RA-01SH)")
+    (date "2023-09-17")
     (company "Missouri S&T Rocket Design Team")
+    (comment 1 "Ariel Pilger")
+  )
+  (junction (at 132.08 102.87) (diameter 0) (color 0 0 0 0)
+  )
+  (no_connect (at 142.24 90.17))
+  (no_connect (at 142.24 92.71))
+  (no_connect (at 142.24 95.25))
+  (wire (pts (xy 132.08 67.31) (xy 132.08 72.39))
+    (stroke (width 0) (type default))
+  )
+  (wire (pts (xy 101.6 85.09) (xy 121.92 85.09))
+    (stroke (width 0) (type default))
+  )
+  (wire (pts (xy 101.6 72.39) (xy 101.6 73.66))
+    (stroke (width 0) (type default))
+  )
+  (wire (pts (xy 101.6 87.63) (xy 121.92 87.63))
+    (stroke (width 0) (type default))
+  )
+  (wire (pts (xy 101.6 90.17) (xy 121.92 90.17))
+    (stroke (width 0) (type default))
+  )
+  (wire (pts (xy 142.24 77.47) (xy 156.21 77.47))
+    (stroke (width 0) (type default))
+  )
+  (wire (pts (xy 101.6 82.55) (xy 101.6 81.28))
+    (stroke (width 0) (type default))
+  )
+  (wire (pts (xy 101.6 82.55) (xy 121.92 82.55))
+    (stroke (width 0) (type default))
+  )
+  (wire (pts (xy 161.29 102.87) (xy 132.08 102.87))
+    (stroke (width 0) (type default))
+  )
+  (wire (pts (xy 161.29 82.55) (xy 161.29 102.87))
+    (stroke (width 0) (type default))
+  )
+  (wire (pts (xy 132.08 102.87) (xy 132.08 105.41))
+    (stroke (width 0) (type default))
+  )
+  (label "MOSI" (at 114.3 85.09 0) (fields_autoplaced)
+    (effects (font (size 1.27 1.27)) (justify left bottom))
+  )
+  (label "SCK" (at 114.3 90.17 0) (fields_autoplaced)
+    (effects (font (size 1.27 1.27)) (justify left bottom))
+  )
+  (label "~{CS}" (at 114.3 82.55 0) (fields_autoplaced)
+    (effects (font (size 1.27 1.27)) (justify left bottom))
+  )
+  (label "MISO" (at 114.3 87.63 0) (fields_autoplaced)
+    (effects (font (size 1.27 1.27)) (justify left bottom))
+  )
+  (hierarchical_label "SCK" (shape input) (at 101.6 90.17 180) (fields_autoplaced)
+    (effects (font (size 1.27 1.27)) (justify right))
+  )
+  (hierarchical_label "MISO" (shape output) (at 101.6 87.63 180) (fields_autoplaced)
+    (effects (font (size 1.27 1.27)) (justify right))
+  )
+  (hierarchical_label "MOSI" (shape input) (at 101.6 85.09 180) (fields_autoplaced)
+    (effects (font (size 1.27 1.27)) (justify right))
+  )
+  (symbol (lib_id "power:GND") (at 132.08 105.41 0) (unit 1)
+    (in_bom yes) (on_board yes) (dnp no) (fields_autoplaced)
+    (property "Reference" "#PWR024" (at 132.08 111.76 0)
+      (effects (font (size 1.27 1.27)) hide)
+    )
+    (property "Value" "GND" (at 132.08 110.49 0)
+      (effects (font (size 1.27 1.27)))
+    )
+    (property "Footprint" "" (at 132.08 105.41 0)
+      (effects (font (size 1.27 1.27)) hide)
+    )
+    (property "Datasheet" "" (at 132.08 105.41 0)
+      (effects (font (size 1.27 1.27)) hide)
+    )
+    (pin "1")
+    (instances
+      (project "FC"
+        (path "/54cce219-8b98-4e71-96c4-f9ee784aa3bc/35031a3a-251a-4009-92bf-5738de5c8c69"
+          (reference "#PWR024") (unit 1)
+        )
+      )
+    )
+  )
+  (symbol (lib_id "RA-01SH:RA-01SH") (at 132.08 87.63 0) (unit 1)
+    (in_bom yes) (on_board yes) (dnp no) (fields_autoplaced)
+    (property "Reference" "U3" (at 134.2741 69.85 0)
+      (effects (font (size 1.27 1.27)) (justify left))
+    )
+    (property "Value" "RA-01SH" (at 134.2741 72.39 0)
+      (effects (font (size 1.27 1.27)) (justify left))
+    )
+    (property "Footprint" "RF_Module:RA-01SH" (at 157.48 97.79 0)
+      (effects (font (size 1.27 1.27)) hide)
+    )
+    (property "Datasheet" "https://docs.ai-thinker.com/_media/lora/docs/ra-01sh_specification.pdf" (at 134.2741 69.85 0)
+      (effects (font (size 1.27 1.27)) (justify left) hide)
+    )
+    (property "Digikey" "https://docs.ai-thinker.com/_media/lora/docs/ra-01sh_specification.pdf" (at 134.2741 72.39 0)
+      (effects (font (size 1.27 1.27)) (justify left) hide)
+    )
+    (pin "1")
+    (pin "10")
+    (pin "11")
+    (pin "12")
+    (pin "13")
+    (pin "14")
+    (pin "15")
+    (pin "16")
+    (pin "2")
+    (pin "3")
+    (pin "4")
+    (pin "5")
+    (pin "6")
+    (pin "7")
+    (pin "8")
+    (pin "9")
+    (instances
+      (project "FC"
+        (path "/54cce219-8b98-4e71-96c4-f9ee784aa3bc/35031a3a-251a-4009-92bf-5738de5c8c69"
+          (reference "U3") (unit 1)
+        )
+      )
+    )
+  )
+  (symbol (lib_id "CONSMA020.062-G:CONSMA020.062-G") (at 161.29 77.47 0) (unit 1)
+    (in_bom yes) (on_board yes) (dnp no) (fields_autoplaced)
+    (property "Reference" "J4" (at 165.1 76.4932 0)
+      (effects (font (size 1.27 1.27)) (justify left))
+    )
+    (property "Value" "CONSMA020.062-G" (at 165.1 79.0332 0)
+      (effects (font (size 1.27 1.27)) (justify left))
+    )
+    (property "Footprint" "CONSMA020.062:CONSMA020.062-G" (at 161.29 77.47 0)
+      (effects (font (size 1.27 1.27)) hide)
+    )
+    (property "Datasheet" " https://linxtechnologies.com/wp/wp-content/uploads/consma020.062-g-ds.pdf" (at 161.29 77.47 0)
+      (effects (font (size 1.27 1.27)) hide)
+    )
+    (property "Digikey" "https://www.digikey.com/en/products/detail/linx-technologies-inc/CONSMA020-062-G/11482822?utm_adgroup=RF%20%26%20RFID&utm_source=google&utm_medium=cpc&utm_campaign=Dynamic%20Search_EN_RLSA_Cart&utm_term=&utm_content=RF%20%26%20RFID&gclid=CjwKCAjwjMiiBhA4EiwAZe6jQ_ICZ5R1fLlqBsg05PucOrzhKWKzfFOsQ26g2j1dcTdAjUSslVJZmhoCegUQAvD_BwE" (at 161.29 77.47 0)
+      (effects (font (size 1.27 1.27)) hide)
+    )
+    (pin "1")
+    (pin "2")
+    (instances
+      (project "FC"
+        (path "/54cce219-8b98-4e71-96c4-f9ee784aa3bc/35031a3a-251a-4009-92bf-5738de5c8c69"
+          (reference "J4") (unit 1)
+        )
+      )
+    )
+  )
+  (symbol (lib_id "Device:R") (at 101.6 77.47 180) (unit 1)
+    (in_bom yes) (on_board yes) (dnp no) (fields_autoplaced)
+    (property "Reference" "R16" (at 104.14 76.2 0)
+      (effects (font (size 1.27 1.27)) (justify right))
+    )
+    (property "Value" "1K" (at 104.14 78.74 0)
+      (effects (font (size 1.27 1.27)) (justify right))
+    )
+    (property "Footprint" "" (at 103.378 77.47 90)
+      (effects (font (size 1.27 1.27)) hide)
+    )
+    (property "Datasheet" "~" (at 101.6 77.47 0)
+      (effects (font (size 1.27 1.27)) hide)
+    )
+    (pin "1")
+    (pin "2")
+    (instances
+      (project "FC"
+        (path "/54cce219-8b98-4e71-96c4-f9ee784aa3bc/35031a3a-251a-4009-92bf-5738de5c8c69"
+          (reference "R16") (unit 1)
+        )
+      )
+    )
+  )
+  (symbol (lib_id "power:+3.3V") (at 132.08 67.31 0) (unit 1)
+    (in_bom yes) (on_board yes) (dnp no) (fields_autoplaced)
+    (property "Reference" "#PWR022" (at 132.08 71.12 0)
+      (effects (font (size 1.27 1.27)) hide)
+    )
+    (property "Value" "+3.3V" (at 132.08 62.23 0)
+      (effects (font (size 1.27 1.27)))
+    )
+    (property "Footprint" "" (at 132.08 67.31 0)
+      (effects (font (size 1.27 1.27)) hide)
+    )
+    (property "Datasheet" "" (at 132.08 67.31 0)
+      (effects (font (size 1.27 1.27)) hide)
+    )
+    (pin "1")
+    (instances
+      (project "FC"
+        (path "/54cce219-8b98-4e71-96c4-f9ee784aa3bc/35031a3a-251a-4009-92bf-5738de5c8c69"
+          (reference "#PWR022") (unit 1)
+        )
+      )
+    )
+  )
+  (symbol (lib_id "power:+3.3V") (at 101.6 72.39 0) (unit 1)
+    (in_bom yes) (on_board yes) (dnp no) (fields_autoplaced)
+    (property "Reference" "#PWR023" (at 101.6 76.2 0)
+      (effects (font (size 1.27 1.27)) hide)
+    )
+    (property "Value" "+3.3V" (at 101.6 67.31 0)
+      (effects (font (size 1.27 1.27)))
+    )
+    (property "Footprint" "" (at 101.6 72.39 0)
+      (effects (font (size 1.27 1.27)) hide)
+    )
+    (property "Datasheet" "" (at 101.6 72.39 0)
+      (effects (font (size 1.27 1.27)) hide)
+    )
+    (pin "1")
+    (instances
+      (project "FC"
+        (path "/54cce219-8b98-4e71-96c4-f9ee784aa3bc/35031a3a-251a-4009-92bf-5738de5c8c69"
+          (reference "#PWR023") (unit 1)
+        )
+      )
+    )
   )
 )
