File: hardware/kicad/hierarchical_sheets/ra-01sh.kicad_sch (KiCad schematic)
At the start: 5 parts, among them J4 CONSMA020.062-G, U6 RA-01SH

Commit message: sync
Parts:
- U6: footprint RF_Module:RA-01SH -> RF_Module:Ai-Thinker-Ra-01-LoRa
Changed lines of the file:
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@@
       (effects (font (size 1.27 1.27)) (justify left))
     )
-    (property "Footprint" "RF_Module:RA-01SH" (at 89.535 93.345 0)
+    (property "Footprint" "RF_Module:Ai-Thinker-Ra-01-LoRa" (at 89.535 93.345 0)
       (effects (font (size 1.27 1.27)) hide)
     )

Commit message: making formatting more consistent
Other:
- moved on the sheet: C7, J4, R16, R17, U6

Commit message: formatting
Parts:
- renumbered U6 to U7
Changed lines of the file:
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@@
   (symbol (lib_id "RA-01SH:RA-01SH") (at 119.38 104.14 0) (unit 1)
     (in_bom yes) (on_board yes) (dnp no) (fields_autoplaced)
-    (property "Reference" "U6" (at 121.5741 86.36 0)
+    (property "Reference" "U7" (at 121.5741 86.36 0)
       (effects (font (size 1.27 1.27)) (justify left))
     )
@@
       (project "FC"
         (path "/54cce219-8b98-4e71-96c4-f9ee784aa3bc/35031a3a-251a-4009-92bf-5738de5c8c69"
-          (reference "U6") (unit 1)
+          (reference "U7") (unit 1)
         )
       )

Commit message: sync
Connections:
- net ANT: now reaches J4.1 (In), U7.1 (ANT)
Changed lines of the file:
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@@
+    (effects (font (size 1.27 1.27)) (justify left bottom))
+  )
+  (label "ANT" (at 130.81 93.98 0) (fields_autoplaced)
     (effects (font (size 1.27 1.27)) (justify left bottom))
   )
@@
     (effects (font (size 1.27 1.27)) (justify right))
   )
+  (netclass_flag "" (length 2.54) (shape round) (at 134.62 93.98 0) (fields_autoplaced)
+    (effects (font (size 1.27 1.27)) (justify left bottom))
+    (property "Netclass" "50_OHM" (at 135.3185 91.44 0)
+      (effects (font (size 1.27 1.27) italic) (justify left))
+    )
+  )
   (symbol (lib_id "power:GND") (at 104.775 85.725 0) (unit 1)

Commit message: work on pcb
Connections:
- net ~{RESET}: now reaches R17.2, U7.4 (~{RESET})
Changed lines of the file:
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@@
+    (effects (font (size 1.27 1.27)) (justify left bottom))
+  )
+  (label "~{RESET}" (at 130.81 101.6 0) (fields_autoplaced)
     (effects (font (size 1.27 1.27)) (justify left bottom))
   )
