File: hardware/kicad/hierarchical_sheets/m10s.kicad_sch (KiCad schematic)
At the start: 4 parts, among them J5 CONSMA020.062-G, U7 MAX-M10S

Commit message: assigned footprints
Parts:
- C1, C2: footprint (none) -> Resistor_SMD:R_0603_1608Metric
Changed lines of the file:
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@@
       (effects (font (size 1.27 1.27)) (justify left))
     )
-    (property "Footprint" "" (at 121.285 64.135 0)
+    (property "Footprint" "Resistor_SMD:R_0603_1608Metric" (at 121.285 64.135 0)
       (effects (font (size 1.27 1.27)) hide)
     )
@@
         )
         (path "/54cce219-8b98-4e71-96c4-f9ee784aa3bc/f2d155c9-a158-4cf0-b4ab-42b0987153ce"
-          (reference "C16") (unit 1)
+          (reference "C9") (unit 1)
         )
       )
@@
         )
         (path "/54cce219-8b98-4e71-96c4-f9ee784aa3bc/f2d155c9-a158-4cf0-b4ab-42b0987153ce"
-          (reference "#PWR041") (unit 1)
+          (reference "#PWR031") (unit 1)
         )
       )
@@
       (effects (font (size 1.27 1.27)) (justify left))
     )
-    (property "Footprint" "" (at 111.76 63.5 0)
+    (property "Footprint" "Resistor_SMD:R_0603_1608Metric" (at 111.76 63.5 0)
       (effects (font (size 1.27 1.27)) hide)
     )
@@
         )
         (path "/54cce219-8b98-4e71-96c4-f9ee784aa3bc/f2d155c9-a158-4cf0-b4ab-42b0987153ce"
-          (reference "C15") (unit 1)
+          (reference "C8") (unit 1)
         )
       )
@@
         )
         (path "/54cce219-8b98-4e71-96c4-f9ee784aa3bc/f2d155c9-a158-4cf0-b4ab-42b0987153ce"
-          (reference "#PWR040") (unit 1)
+          (reference "#PWR030") (unit 1)
         )
       )
@@
   (symbol (lib_id "power:GND") (at 139.065 118.745 0) (unit 1)
     (in_bom yes) (on_board yes) (dnp no) (fields_autoplaced)
-    (property "Reference" "#PWR038" (at 139.065 125.095 0)
+    (property "Reference" "#PWR032" (at 139.065 125.095 0)
       (effects (font (size 1.27 1.27)) hide)
     )
@@
       (project "FC"
         (path "/54cce219-8b98-4e71-96c4-f9ee784aa3bc/f2d155c9-a158-4cf0-b4ab-42b0987153ce"
-          (reference "#PWR038") (unit 1)
+          (reference "#PWR032") (unit 1)
         )
       )

Commit message: added gps integration manual and note on gps schematic
Other:
- note added: "pg 71 of integration manual: Might want to add the components for an active antenna supply. Looks like active antennas are much easier to find."
Changed lines of the file:
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@@
     (stroke (width 0) (type default))
+  )
+  (text "pg 71 of integration manual: \nMight want to add the components for an active antenna\nsupply. Looks like active antennas are much easier to find. "
+    (at 164.465 81.28 0)
+    (effects (font (size 1.27 1.27)) (justify left bottom))
   )
   (text "Addr: 0x42" (at 116.84 116.84 0)

Commit message: formatting
Parts:
- renumbered U7 to U8
Changed lines of the file:
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@@
   (symbol (lib_id "RF_GPS:MAX-M10S") (at 139.065 94.615 0) (unit 1)
     (in_bom yes) (on_board yes) (dnp no) (fields_autoplaced)
-    (property "Reference" "U7" (at 141.2591 111.76 0)
+    (property "Reference" "U8" (at 141.2591 111.76 0)
       (effects (font (size 1.27 1.27)) (justify left))
     )
@@
       (project "FC"
         (path "/54cce219-8b98-4e71-96c4-f9ee784aa3bc/f2d155c9-a158-4cf0-b4ab-42b0987153ce"
-          (reference "U7") (unit 1)
+          (reference "U8") (unit 1)
         )
       )

Commit message: formatting / exported pdf
Other:
- title: SRAD-FC -> GPS (M10S)
Changed lines of the file:
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@@
   (paper "USLetter")
   (title_block
-    (title "SRAD-FC")
+    (title "GPS (M10S)")
     (company "Missouri S&T Rocket Design Team")
     (comment 1 "Riley Kyle")
@@
   )
   (symbol (lib_id "RF_GPS:MAX-M10S") (at 139.065 94.615 0) (unit 1)
-    (in_bom yes) (on_board yes) (dnp no) (fields_autoplaced)
-    (property "Reference" "U8" (at 141.2591 111.76 0)
+    (in_bom yes) (on_board yes) (dnp no)
+    (property "Reference" "U8" (at 147.32 74.295 0)
       (effects (font (size 1.27 1.27)) (justify left))
     )
-    (property "Value" "MAX-M10S" (at 141.2591 114.3 0)
+    (property "Value" "MAX-M10S" (at 147.32 76.835 0)
       (effects (font (size 1.27 1.27)) (justify left))
     )

Commit message: GPS Ant. SN
Parts:
- added C25: GRM155R71C103KA01J, Capacitor_SMD:C_01005_0402Metric, symbol Device:C
- added L1: LQW15AN27NJ00D, Inductor_SMD:L_0402_1005Metric, symbol Device:L
- added R30: 10R, Resistor_SMD:R_0603_1608Metric, symbol Device:R
Connections:
- net GND: now also C25.2
- net at J5.1 (In), U8.11 (RF_IN): now also L1.2
- net at U8.14 (VCC_RF): now also R30.1
- new net: C25.1, L1.1, R30.2
- no-connect marks 10 -> 9
Other:
- note removed: "pg 71 of integration manual: Might want to add the components for an active antenna supply. Looks like active antennas are much easier to find."
- moved on the sheet: J5
Changed lines of the file:
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@@
   (junction (at 136.525 76.835) (diameter 0) (color 0 0 0 0)
   )
+  (junction (at 167.64 67.31) (diameter 0) (color 0 0 0 0)
+  )
   (junction (at 133.985 73.025) (diameter 0) (color 0 0 0 0)
   )
@@
   )
   (junction (at 121.285 68.58) (diameter 0) (color 0 0 0 0)
+  )
+  (junction (at 167.64 94.615) (diameter 0) (color 0 0 0 0)
   )
   (junction (at 133.985 76.835) (diameter 0) (color 0 0 0 0)
@@
   (no_connect (at 123.825 107.315))
   (no_connect (at 154.305 89.535))
-  (no_connect (at 144.145 76.835))
   (no_connect (at 123.825 102.235))
   (no_connect (at 123.825 104.775))
@@
   (no_connect (at 139.065 76.835))
   (no_connect (at 154.305 102.235))
-  (wire (pts (xy 161.925 94.615) (xy 154.305 94.615))
+  (wire (pts (xy 182.245 94.615) (xy 167.64 94.615))
+    (stroke (width 0) (type default))
+  )
+  (wire (pts (xy 222.25 67.31) (xy 184.785 67.31))
     (stroke (width 0) (type default))
   )
@@
     (stroke (width 0) (type default))
   )
+  (wire (pts (xy 167.64 94.615) (xy 154.305 94.615))
+    (stroke (width 0) (type default))
+  )
+  (wire (pts (xy 144.145 67.31) (xy 144.145 76.835))
+    (stroke (width 0) (type default))
+  )
+  (wire (pts (xy 167.64 90.805) (xy 167.64 94.615))
+    (stroke (width 0) (type default))
+  )
   (wire (pts (xy 111.76 66.04) (xy 111.76 68.58))
     (stroke (width 0) (type default))
@@
     (stroke (width 0) (type default))
   )
+  (wire (pts (xy 222.25 69.85) (xy 222.25 67.31))
+    (stroke (width 0) (type default))
+  )
+  (wire (pts (xy 167.64 67.31) (xy 167.64 83.185))
+    (stroke (width 0) (type default))
+  )
   (wire (pts (xy 111.76 59.69) (xy 111.76 60.96))
     (stroke (width 0) (type default))
@@
     (stroke (width 0) (type default))
   )
+  (wire (pts (xy 151.13 67.31) (xy 144.145 67.31))
+    (stroke (width 0) (type default))
+  )
   (wire (pts (xy 139.065 118.745) (xy 139.065 112.395))
     (stroke (width 0) (type default))
@@
     (stroke (width 0) (type default))
   )
+  (wire (pts (xy 139.065 118.745) (xy 187.325 118.745))
+    (stroke (width 0) (type default))
+  )
   (wire (pts (xy 121.285 59.69) (xy 121.285 61.595))
     (stroke (width 0) (type default))
@@
     (stroke (width 0) (type default))
   )
-  (wire (pts (xy 167.005 99.695) (xy 167.005 118.745))
-    (stroke (width 0) (type default))
-  )
-  (wire (pts (xy 167.005 118.745) (xy 139.065 118.745))
+  (wire (pts (xy 167.64 67.31) (xy 158.75 67.31))
+    (stroke (width 0) (type default))
+  )
+  (wire (pts (xy 187.325 99.695) (xy 187.325 118.745))
     (stroke (width 0) (type default))
   )
@@
     (stroke (width 0) (type default))
   )
+  (wire (pts (xy 167.64 67.31) (xy 177.165 67.31))
+    (stroke (width 0) (type default))
+  )
   (wire (pts (xy 133.985 59.69) (xy 133.985 73.025))
     (stroke (width 0) (type default))
-  )
-  (text "pg 71 of integration manual: \nMight want to add the components for an active antenna\nsupply. Looks like active antennas are much easier to find. "
-    (at 164.465 81.28 0)
-    (effects (font (size 1.27 1.27)) (justify left bottom))
   )
   (text "Addr: 0x42" (at 116.84 116.84 0)
@@
   (hierarchical_label "SDA" (shape bidirectional) (at 111.76 92.075 180) (fields_autoplaced)
     (effects (font (size 1.27 1.27)) (justify right))
+  )
+  (symbol (lib_id "power:GND") (at 222.25 69.85 0) (unit 1)
+    (in_bom yes) (on_board yes) (dnp no) (fields_autoplaced)
+    (property "Reference" "#PWR063" (at 222.25 76.2 0)
+      (effects (font (size 1.27 1.27)) hide)
+    )
+    (property "Value" "GND" (at 222.25 74.93 0)
+      (effects (font (size 1.27 1.27)))
+    )
+    (property "Footprint" "" (at 222.25 69.85 0)
+      (effects (font (size 1.27 1.27)) hide)
+    )
+    (property "Datasheet" "" (at 222.25 69.85 0)
+      (effects (font (size 1.27 1.27)) hide)
+    )
+    (pin "1")
+    (instances
+      (project "FC"
+        (path "/54cce219-8b98-4e71-96c4-f9ee784aa3bc/f2d155c9-a158-4cf0-b4ab-42b0987153ce"
+          (reference "#PWR063") (unit 1)
+        )
+      )
+    )
   )
   (symbol (lib_id "Device:C_Small") (at 121.285 64.135 0) (unit 1)
@@
     )
   )
-  (symbol (lib_id "CONSMA020.062-G:CONSMA020.062-G") (at 167.005 94.615 0) (unit 1)
-    (in_bom yes) (on_board yes) (dnp no) (fields_autoplaced)
-    (property "Reference" "J5" (at 170.18 93.6382 0)
-      (effects (font (size 1.27 1.27)) (justify left))
-    )
-    (property "Value" "CONSMA020.062-G" (at 170.18 96.1782 0)
-      (effects (font (size 1.27 1.27)) (justify left))
-    )
-    (property "Footprint" "CONSMA020.062:CONSMA020.062-G" (at 167.005 94.615 0)
-      (effects (font (size 1.27 1.27)) hide)
-    )
-    (property "Datasheet" " https://linxtechnologies.com/wp/wp-content/uploads/consma020.062-g-ds.pdf" (at 167.005 94.615 0)
-      (effects (font (size 1.27 1.27)) hide)
-    )
-    (property "Digikey" "https://www.digikey.com/en/products/detail/linx-technologies-inc/CONSMA020-062-G/11482822?utm_adgroup=RF%20%26%20RFID&utm_source=google&utm_medium=cpc&utm_campaign=Dynamic%20Search_EN_RLSA_Cart&utm_term=&utm_content=RF%20%26%20RFID&gclid=CjwKCAjwjMiiBhA4EiwAZe6jQ_ICZ5R1fLlqBsg05PucOrzhKWKzfFOsQ26g2j1dcTdAjUSslVJZmhoCegUQAvD_BwE" (at 167.005 94.615 0)
+  (symbol (lib_id "Device:R") (at 154.94 67.31 90) (unit 1)
+    (in_bom yes) (on_board yes) (dnp no) (fields_autoplaced)
+    (property "Reference" "R30" (at 154.94 60.96 90)
+      (effects (font (size 1.27 1.27)))
+    )
+    (property "Value" "10R" (at 154.94 63.5 90)
+      (effects (font (size 1.27 1.27)))
+    )
+    (property "Footprint" "Resistor_SMD:R_0603_1608Metric" (at 154.94 69.088 90)
+      (effects (font (size 1.27 1.27)) hide)
+    )
+    (property "Datasheet" "~" (at 154.94 67.31 0)
+      (effects (font (size 1.27 1.27)) hide)
+    )
+    (pin "1")
+    (pin "2")
+    (instances
+      (project "FC"
+        (path "/54cce219-8b98-4e71-96c4-f9ee784aa3bc/f2d155c9-a158-4cf0-b4ab-42b0987153ce"
+          (reference "R30") (unit 1)
+        )
+      )
+    )
+  )
+  (symbol (lib_id "CONSMA020.062-G:CONSMA020.062-G") (at 187.325 94.615 0) (unit 1)
+    (in_bom yes) (on_board yes) (dnp no) (fields_autoplaced)
+    (property "Reference" "J5" (at 190.5 93.6382 0)
+      (effects (font (size 1.27 1.27)) (justify left))
+    )
+    (property "Value" "CONSMA020.062-G" (at 190.5 96.1782 0)
+      (effects (font (size 1.27 1.27)) (justify left))
+    )
+    (property "Footprint" "CONSMA020.062:CONSMA020.062-G" (at 187.325 94.615 0)
+      (effects (font (size 1.27 1.27)) hide)
+    )
+    (property "Datasheet" " https://linxtechnologies.com/wp/wp-content/uploads/consma020.062-g-ds.pdf" (at 187.325 94.615 0)
+      (effects (font (size 1.27 1.27)) hide)
+    )
+    (property "Digikey" "https://www.digikey.com/en/products/detail/linx-technologies-inc/CONSMA020-062-G/11482822?utm_adgroup=RF%20%26%20RFID&utm_source=google&utm_medium=cpc&utm_campaign=Dynamic%20Search_EN_RLSA_Cart&utm_term=&utm_content=RF%20%26%20RFID&gclid=CjwKCAjwjMiiBhA4EiwAZe6jQ_ICZ5R1fLlqBsg05PucOrzhKWKzfFOsQ26g2j1dcTdAjUSslVJZmhoCegUQAvD_BwE" (at 187.325 94.615 0)
       (effects (font (size 1.27 1.27)) hide)
     )
@@
         )
       )
+    )
+  )
+  (symbol (lib_id "Device:L") (at 167.64 86.995 0) (unit 1)
+    (in_bom yes) (on_board yes) (dnp no) (fields_autoplaced)
+    (property "Reference" "L1" (at 168.91 85.725 0)
+      (effects (font (size 1.27 1.27)) (justify left))
+    )
+    (property "Value" "LQW15AN27NJ00D" (at 168.91 88.265 0)
+      (effects (font (size 1.27 1.27)) (justify left))
+    )
+    (property "Footprint" "Inductor_SMD:L_0402_1005Metric" (at 167.64 86.995 0)
+      (effects (font (size 1.27 1.27)) hide)
+    )
+    (property "Datasheet" "https://search.murata.co.jp/Ceramy/image/img/P02/JELF243A-0050.pdf" (at 167.64 86.995 0)
+      (effects (font (size 1.27 1.27)) hide)
+    )
+    (property "Digikey" "https://www.digikey.com/en/products/detail/murata-electronics/LQW15AN27NJ00D/584360" (at 167.64 86.995 0)
+      (effects (font (size 1.27 1.27)) hide)
+    )
+    (pin "1")
+    (pin "2")
+    (instances
+      (project "FC"
+        (path "/54cce219-8b98-4e71-96c4-f9ee784aa3bc/f2d155c9-a158-4cf0-b4ab-42b0987153ce"
+          (reference "L1") (unit 1)
+        )
+      )
+    )
+  )
+  (symbol (lib_id "Device:C") (at 180.975 67.31 90) (unit 1)
+    (in_bom yes) (on_board yes) (dnp no) (fields_autoplaced)
+    (property "Reference" "C25" (at 180.975 59.69 90)
+      (effects (font (size 1.27 1.27)))
+    )
+    (property "Value" "GRM155R71C103KA01J" (at 180.975 62.23 90)
+      (effects (font (size 1.27 1.27)))
+    )
+    (property "Footprint" "Capacitor_SMD:C_01005_0402Metric" (at 184.785 66.3448 0)
+      (effects (font (size 1.27 1.27)) hide)
+    )
+    (property "Datasheet" "https://search.murata.co.jp/Ceramy/image/img/A01X/G101/ENG/GRM155R71C103KA01-01.pdf" (at 180.975 67.31 0)
+      (effects (font (size 1.27 1.27)) hide)
+    )
+    (property "Digikey" "https://www.digikey.com/en/products/detail/murata-electronics/GRM155R71C103KA01J/2610890" (at 180.975 67.31 90)
+      (effects (font (size 1.27 1.27)) hide)
+    )
+    (pin "1")
+    (pin "2")
+    (instances
+      (project "FC"
+        (path "/54cce219-8b98-4e71-96c4-f9ee784aa3bc/f2d155c9-a158-4cf0-b4ab-42b0987153ce"
+          (reference "C25") (unit 1)
+        )
+      )

Commit message: pcb work started
Parts:
- C25: footprint Capacitor_SMD:C_01005_0402Metric -> Capacitor_SMD:C_0402_1005Metric
Changed lines of the file:
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@@
       (effects (font (size 1.27 1.27)))
     )
-    (property "Footprint" "Capacitor_SMD:C_01005_0402Metric" (at 184.785 66.3448 0)
+    (property "Footprint" "Capacitor_SMD:C_0402_1005Metric" (at 184.785 66.3448 0)
       (effects (font (size 1.27 1.27)) hide)
     )

Commit message: sync
Connections:
- net RF_IN: now reaches J5.1 (In), L1.2, U8.11 (RF_IN)
Changed lines of the file:
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@@
+    (effects (font (size 1.27 1.27)) (justify left bottom))
+  )
+  (label "RF_IN" (at 158.115 94.615 0) (fields_autoplaced)
     (effects (font (size 1.27 1.27)) (justify left bottom))
   )
@@
     (effects (font (size 1.27 1.27)) (justify right))
   )
+  (netclass_flag "" (length 2.54) (shape round) (at 172.085 94.615 0) (fields_autoplaced)
+    (effects (font (size 1.27 1.27)) (justify left bottom))
+    (property "Netclass" "50_OHM" (at 172.7835 92.075 0)
+      (effects (font (size 1.27 1.27) italic) (justify left))
+    )
+  )
   (symbol (lib_id "power:GND") (at 222.25 69.85 0) (unit 1)
