File: hardware/kicad/hierarchical_sheets/m10s.kicad_sch (KiCad schematic)
At the start: 7 parts, among them J5 CONSMA020.062-G, U8 MAX-M10S

Commit message: sync
Parts:
- U8: Digikey (none) -> https://www.digikey.com/en/products/detail/u-blox/MAX-M10S-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
Changed lines of the file:
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@@
+      (effects (font (size 1.27 1.27)) hide)
+    )
+    (property "Digikey" "https://www.digikey.com/en/products/detail/u-blox/MAX-M10S-00B/15712906" (at 139.065 94.615 0)
       (effects (font (size 1.27 1.27)) hide)
     )

Commit message: appended .off to old files
Parts:
- renumbered C1 to C8, C2 to C9
