File: hardware/kicad/hierarchical_sheets/atmega32u4.kicad_sch (KiCad schematic)
At the start: 41 parts, among them J6 0475900001, J7 TC2030, U12 ATmega32U4-A, Y1 16MHz

Commit message: massive routing progress
Connections:
- net CH1_FIRE: now also U12.8 (PB0); no longer U12.22 (PD5)
- net CH2_FIRE: now also U12.22 (PD5); no longer U12.8 (PB0)
Changed lines of the file:
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@@
     (effects (font (size 1.27 1.27)) (justify left bottom))
   )
-  (label "CH2_FIRE" (at 114.935 57.785 0) (fields_autoplaced)
+  (label "CH2_FIRE" (at 114.935 100.965 0) (fields_autoplaced)
     (effects (font (size 0.63 0.63)) (justify left bottom))
   )
@@
     (effects (font (size 1.27 1.27)) (justify left bottom))
   )
-  (label "CH1_FIRE" (at 114.935 100.965 0) (fields_autoplaced)
+  (label "CH1_FIRE" (at 116.205 57.785 0) (fields_autoplaced)
     (effects (font (size 0.63 0.63)) (justify left bottom))
   )
@@
     (effects (font (size 1.27 1.27)) (justify left))
   )
-  (hierarchical_label "CH2_FIRE" (shape output) (at 125.73 57.785 0) (fields_autoplaced)
+  (hierarchical_label "CH2_FIRE" (shape output) (at 125.73 100.965 0) (fields_autoplaced)
     (effects (font (size 1.27 1.27)) (justify left))
   )
@@
     (effects (font (size 1.27 1.27)) (justify left))
   )
-  (hierarchical_label "CH1_FIRE" (shape output) (at 125.73 100.965 0) (fields_autoplaced)
-    (effects (font (size 1.27 1.27)) (justify left))
-  )
+  (hierarchical_label "CH1_FIRE" (shape output) (at 125.73 57.785 0) (fields_autoplaced)
+    (effects (font (size 1.27 1.27)) (justify left))
+  )

Commit message: dont break plz
Connections:
- net CH1_DETECT: now also U12.28 (PB4); no longer U12.30 (PB6)
- net CH2_DETECT: now also U12.30 (PB6); no longer U12.28 (PB4)
Changed lines of the file:
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@@
     (effects (font (size 1.27 1.27)) (justify left bottom))
   )
-  (label "CH1_DETECT" (at 114.935 73.025 0) (fields_autoplaced)
+  (label "CH1_DETECT" (at 114.935 67.945 0) (fields_autoplaced)
     (effects (font (size 0.63 0.63)) (justify left bottom))
   )
@@
     (effects (font (size 0.63 0.63)) (justify left bottom))
   )
-  (label "CH2_DETECT" (at 114.935 67.945 0) (fields_autoplaced)
+  (label "CH2_DETECT" (at 114.935 73.025 0) (fields_autoplaced)
     (effects (font (size 0.63 0.63)) (justify left bottom))
   )
@@
     (effects (font (size 1.27 1.27)) (justify left))
   )
-  (hierarchical_label "CH2_DETECT" (shape input) (at 125.73 67.945 0) (fields_autoplaced)
+  (hierarchical_label "CH2_DETECT" (shape input) (at 125.73 73.025 0) (fields_autoplaced)
     (effects (font (size 1.27 1.27)) (justify left))
   )
@@
     (effects (font (size 1.27 1.27)) (justify left))
   )
-  (hierarchical_label "CH1_DETECT" (shape input) (at 125.73 73.025 0) (fields_autoplaced)
+  (hierarchical_label "CH1_DETECT" (shape input) (at 125.73 67.945 0) (fields_autoplaced)
     (effects (font (size 1.27 1.27)) (justify left))
   )

Commit message: cs lines
Connections:
- net ~{BAROMETER_CS}: now also U12.37 (PF6); no longer U12.41 (PF0)
- net ~{FRAM_CS}: now also U12.41 (PF0); no longer U12.37 (PF6)
- net ~{FRAM_HOLD}: now also U12.40 (PF1); no longer U12.36 (PF7)
- net ~{IMU_CS}: now also U12.36 (PF7); no longer U12.40 (PF1)
Changed lines of the file:
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@@
     (effects (font (size 1.27 1.27)) (justify left))
   )
-  (hierarchical_label "~{IMU_CS}" (shape output) (at 125.73 121.285 0) (fields_autoplaced)
+  (hierarchical_label "~{IMU_CS}" (shape output) (at 125.73 131.445 0) (fields_autoplaced)
     (effects (font (size 1.27 1.27)) (justify left))
   )
@@
     (effects (font (size 1.27 1.27)) (justify left))
   )
-  (hierarchical_label "~{FRAM_CS}" (shape output) (at 125.73 128.905 0) (fields_autoplaced)
+  (hierarchical_label "~{FRAM_CS}" (shape output) (at 125.73 118.745 0) (fields_autoplaced)
     (effects (font (size 1.27 1.27)) (justify left))
   )
-  (hierarchical_label "~{FRAM_HOLD}" (shape output) (at 125.73 131.445 0) (fields_autoplaced)
+  (hierarchical_label "~{FRAM_HOLD}" (shape output) (at 125.73 121.285 0) (fields_autoplaced)
     (effects (font (size 1.27 1.27)) (justify left))
   )
@@
     (effects (font (size 1.27 1.27)) (justify left))
   )
-  (hierarchical_label "~{BAROMETER_CS}" (shape output) (at 125.73 118.745 0) (fields_autoplaced)
+  (hierarchical_label "~{BAROMETER_CS}" (shape output) (at 125.73 128.905 0) (fields_autoplaced)
     (effects (font (size 1.27 1.27)) (justify left))
   )

Commit message: finished routing
Parts:
- removed TP1, TP10, TP11, TP2, TP3, TP4, TP5, TP6, TP7, TP8, TP9: TestPoint, TestPoint:TestPoint_Pad_D1.5mm, symbol Connector:TestPoint
Connections:
- net ~{BAROMETER_CS}: now also U12.38 (PF5); no longer U12.37 (PF6)
- net ~{HG_ACCEL_CS}: now also U12.36 (PF7); no longer U12.39 (PF4)
- net ~{IMU_CS}: now also U12.37 (PF6); no longer U12.36 (PF7)
- net ~{TELEMETRY_CS}: now also U12.39 (PF4); no longer U12.38 (PF5)
Other:
- note removed: "TEST POINTS"

Commit message: added gnd pour under rf
Connections:
- net ~{HG_ACCEL_CS}: now also U12.37 (PF6); no longer U12.36 (PF7)
- net ~{IMU_CS}: now also U12.36 (PF7); no longer U12.37 (PF6)
Changed lines of the file:
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@@
     (effects (font (size 1.27 1.27)) (justify left))
   )
-  (hierarchical_label "~{IMU_CS}" (shape output) (at 125.73 128.905 0) (fields_autoplaced)
+  (hierarchical_label "~{IMU_CS}" (shape output) (at 125.73 131.445 0) (fields_autoplaced)
     (effects (font (size 1.27 1.27)) (justify left))
   )
@@
     (effects (font (size 1.27 1.27)) (justify left))
   )
-  (hierarchical_label "~{HG_ACCEL_CS}" (shape output) (at 125.73 131.445 0) (fields_autoplaced)
+  (hierarchical_label "~{HG_ACCEL_CS}" (shape output) (at 125.73 128.905 0) (fields_autoplaced)
     (effects (font (size 1.27 1.27)) (justify left))
   )
