File: hardware/kicad/hierarchical_sheets/kx134-1211.kicad_sch (KiCad schematic)
At the start: 4 parts, among them U4 KX134-1211

Commit message: formatting
Other:
- title: SRAD-FC -> High G Accelerometer (KX134-1211)
Changed lines of the file:
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@@
   (paper "USLetter")
   (title_block
-    (title "SRAD-FC")
+    (title "High G Accelerometer (KX134-1211)")
     (company "Missouri S&T Rocket Design Team")
     (comment 1 "Skye Watson")

Commit message: sync
Parts:
- U4: Digikey (none) -> https://www.digikey.com/en/products/detail/rohm-semiconduct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
Changed lines of the file:
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@@
+      (effects (font (size 1.27 1.27)) hide)
+    )
+    (property "Digikey" "https://www.digikey.com/en/products/detail/rohm-semiconductor/KX134-1211/10488055" (at 132.715 99.06 0)
       (effects (font (size 1.27 1.27)) hide)
     )
